File: ele/MainBoard/MainBoard.brd (EAGLE design)
At the start: 101.6 x 61 mm, 85 parts, among them Q1 AO3401ASOP-8_EP_5.0X5.0X1.27P, Q3 AO3401ASOP-8_EP_5.0X5.0X1.27P, SW0 TL3342F160QG/TR, SW1 TL3342F160QG/TR, SW2 TL3342F160QG/TR, SW3 TL3342F160QG/TR, U2 STM32F103VCT6, X1 POWER_IN, X2 POWER_IN, X4 POWER_IN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

Commit message: MainBoardSCH: Add all required peripheries to STM MCU, finish encoder pinouts
TODO:
- fix motor PWMs output for DRV8833
- add ESP32 connectors
- add ultrasonic connectors
- add servo connectors
Parts:
- added BAT_HOLDER: CR2032CR2032-BS-6-1, CR2032-circle:SMD-BAT-CR2032-BS-6-1
- added C19: 2,2uf, resistor:C0805
- added C21: 100nf, resistor:C0402
- added IM1: STEPDOWN, StepDown:STEPDOWN
- added JP10: IM1_2, pinhead:1X02
- added JP11: IM1_EN, pinhead:1X01
- added JP15: M2, pinhead:1X06
- added JP17: M1, pinhead:1X06
- added SJ1, SJ2: (no value), jumper:SJ_2
- added X0: POWER_IN, con-wago-508:W237-132
- added X3: M3B, con-wago-508:W237-132
- added Y1: 3215_2P, SMD3215_2P:SMD-3215_2P
- JP12: value (none) -> M3
- JP6: value (none) -> M4
- U$1: value CR2032 -> DRV8833HTSSOP; device CR2032:CH075 -> texas-cc2541:HTSSOP
- X1: value POWER_IN -> M1B
- X2: value POWER_IN -> M2B
- X4: value POWER_IN -> M4B
- moved JP12 392.6 mm to (-35.6, -325.1)
- moved JP6 380.6 mm to (-35.6, -317.5)
- moved X4 274.7 mm to (-40.6, -193.0), turned to 0 degrees
- moved U$1 17.0 mm to (-33.0, -203.2)
Connections:
- removed net ENC_1A: U2.40
- removed net ENC_1B: U2.42
- removed net ENC_2A: U2.77
- removed net ENC_2B: U2.89
- removed net ENC_3A: U2.31
- removed net ENC_3B: U2.32
- removed net ENC_4A: U2.59
- removed net ENC_4B: U2.60
- removed net ENC_A1: JP12.3
- removed net ENC_A2: JP6.4
- removed net ENC_B1: JP12.4
- removed net ENC_B2: JP6.3
- removed net IO9_NC2: U$9.NFAULT
- removed net PWM_A0: U$9.AIN1
- removed net PWM_A1: U$9.AIN2
- removed net PWM_B0: U$9.BIN1
- removed net PWM_B1: U$9.BIN2
- removed net SLEEP: IM6.24, U$9.NSLEEP
- new net 5V_2: JP10.1
- new net ENC12PWR: JP12.2, JP15.2, JP17.2, JP6.2, SJ1.2, SJ2.2
- new net ENC1A: JP17.3, U2.40
- new net ENC1B: JP17.4, U2.42
- new net ENC2A: JP15.3, U2.77
- new net ENC2B: JP15.4, U2.89
- new net ENC3A: JP12.3, U2.31
- new net ENC3B: JP12.4, U2.32
- new net ENC4A: JP6.3, U2.59
- new net ENC4B: JP6.4, U2.60
- new net M3A: JP12.1, U$1.AOUT1, X3.1
- new net M3B: JP12.6, U$1.AOUT2, X3.2
- new net M4A: JP6.1, U$1.BOUT1, X4.2
- new net M4B: JP6.6, U$1.BOUT2, X4.1
- new net N$3: IM6.24
- new net N$4: IM6.25
- new net N$6: C19.1, U$1.VINT
- new net N$7: C21.1, U$1.VCP
- new net N$8: IM1.EN, JP11.1
- new net OSC32_IN: U2.8
- new net OSC32_OUT: U2.9
- new net _DRIVER_FAULT: U$1.NFAULT, U$9.NFAULT, U2.41
- net +3V3: now also SJ1.1, SJ2.1, U$1.NSLEEP, U$9.NSLEEP
- net +5V: now also IM1.OUT, JP10.2, SJ1.3, SJ2.3; no longer JP12.5, JP6.2
- net 3,3!KNOFLIK: now also BAT_HOLDER.VBAT; no longer U$1.+
- net BAT1: now also X0.2; no longer X4.2
- net DIR_1/2: now also U$9.AIN2
- net DIR_2/1: now also U$9.BIN2
- net DIR_3/4: now also U$1.AIN2
- net DIR_4/3: now also U$1.BIN2
- net GND: now also BAT_HOLDER.VSS, C19.2, IM1.GND, JP12.5, JP15.5, JP17.5, U$1.AISEN, U$1.BISEN, U$1.GND, X0.1; no longer JP12.2, U$1.-, X4.1
- net M1A: now also JP17.1; no longer JP12.6
- net M1B: now also JP17.6; no longer JP12.1
- net M2A: now also JP15.1, X2.1; no longer JP6.1, X2.2
- net M2B: now also JP15.6, X2.2; no longer JP6.6, X2.1
- net PWM1: now also U$9.AIN1
- net PWM2: now also U$9.BIN1
- net PWM3: now also U$1.AIN1
- net PWM4: now also U$1.BIN1
- net VCC: now also C21.2, IM1.IN, U$1.VM
Routing:
- net ENC_A1: track 54.5 -> 0.00 mm
- net ENC_A2: track 51.3 -> 0.00 mm
- net ENC_B2: track 50.6 -> 0.00 mm
- net ENC_B1: track 50.0 -> 0.00 mm
- net PWM_B0: track 39.8 -> 0.00 mm, vias 1 -> 0
- net PWM2: track 0.00 -> 39.8 mm, vias 0 -> 1
- net PWM_A1: track 39.6 -> 0.00 mm, vias 1 -> 0
- net DIR_1/2: track 0.00 -> 39.6 mm, vias 0 -> 1
- net PWM_B1: track 39.0 -> 0.00 mm, vias 1 -> 0
- net DIR_2/1: track 0.00 -> 39.0 mm, vias 0 -> 1
- net PWM_A0: track 38.5 -> 0.00 mm, vias 1 -> 0
- net PWM1: track 0.00 -> 38.5 mm, vias 0 -> 1
- net SLEEP: track 36.2 -> 0.00 mm, vias 1 -> 0
- net +5V: track 99.0 -> 66.1 mm
Other:
- board size 101.6 x 61 mm -> 100 x 100 mm
