File: ele/MainBoard/RBCX-MainBoard.brd (EAGLE design)
At the start: 100 x 100 mm, 336 parts, among them IC1 DRV8833PWP, IC10 INA180A4, IC11 AMS1117-3.3, IC2 INA180A4, IC3 INA180A4, IC4 DRV8833PWP, IC5 INA180A4, IC6 INA180A4, IC7 INA180A4, IC8 INA180A4, IC9 INA180A4, Q1 CHOOSE_ME, Q10 CHOOSE_ME, Q2 CHOOSE_ME, Q3 CHOOSE_ME, Q4 CHOOSE_ME, Q5 CHOOSE_ME, Q6 CHOOSE_ME, Q7 CHOOSE_ME, Q8 CHOOSE_ME, Q9 CHOOSE_ME, U1 STM32F103VCT6, X0 POWER_IN, X1 M3B, X2 M4B, X3 M3B, X4 M4B, X5 POWER_OUT, Y1 3215_2P, Y2 5032/2P

Commit message: MainBoardSCH: Add ESP UART and expander uart connector
Parts:
- added JP58: ESP_UART, pinhead:1X03
- added JP59: EXPANDER_UART, pinhead:1X03
- added R127, R128, R129, R130: 180R, rcl_upravena:R0603
Connections:
- new net ESP-UART-RX: JP58.1, R127.2
- new net ESP-UART-TX: JP58.2, R128.2
- new net EXPANDER-UART-RX: JP59.1, R129.2
- new net EXPANDER-UART-TX: JP59.2, R130.2
- net ESP_COM_RX: now also R129.1
- net ESP_COM_TX: now also R130.1
- net GND: now also JP58.3, JP59.3
- net UART_RX: now also R127.1
- net UART_TX: now also R128.1
Changed lines of the file:
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@@
 <attribute name="VALUE" x="-149.69" y="847.33" size="1.27" layer="27"/>
+</element>
+<element name="JP58" library="pinhead" library_urn="urn:adsk.eagle:library:325" package="1X03" package3d_urn="urn:adsk.eagle:package:22458/2" value="ESP_UART" x="-147.32" y="857.25" smashed="yes">
+<attribute name="NAME" x="-151.2062" y="859.0788" size="1.27" layer="25" ratio="10"/>
+<attribute name="POPULARITY" value="92" x="-147.32" y="-1555.75" size="1.778" layer="27" display="off"/>
+<attribute name="VALUE" x="-151.13" y="854.075" size="1.27" layer="27"/>
+</element>
+<element name="R127" library="rcl_upravena" package="R0603" value="180R" x="-149.86" y="-1554.48" smashed="yes">
+<attribute name="NAME" x="-150.495" y="-1553.845" size="1.27" layer="25"/>
+<attribute name="VALUE" x="-150.495" y="-1556.385" size="1.27" layer="27"/>
+</element>
+<element name="R128" library="rcl_upravena" package="R0603" value="180R" x="-149.86" y="-1559.56" smashed="yes">
+<attribute name="NAME" x="-150.495" y="-1558.925" size="1.27" layer="25"/>
+<attribute name="VALUE" x="-150.495" y="-1561.465" size="1.27" layer="27"/>
+</element>
+<element name="JP59" library="pinhead" library_urn="urn:adsk.eagle:library:325" package="1X03" package3d_urn="urn:adsk.eagle:package:22458/2" value="EXPANDER_UART" x="-147.32" y="864.87" smashed="yes">
+<attribute name="NAME" x="-151.2062" y="866.6988" size="1.27" layer="25" ratio="10"/>
+<attribute name="POPULARITY" value="92" x="-147.32" y="-1565.91" size="1.778" layer="27" display="off"/>
+<attribute name="VALUE" x="-151.13" y="861.695" size="1.27" layer="27"/>
+</element>
+<element name="R129" library="rcl_upravena" package="R0603" value="180R" x="-149.86" y="871.22" smashed="yes">
+<attribute name="NAME" x="-150.495" y="871.855" size="1.27" layer="25"/>
+<attribute name="VALUE" x="-150.495" y="869.315" size="1.27" layer="27"/>
+</element>
+<element name="R130" library="rcl_upravena" package="R0603" value="180R" x="-149.86" y="876.3" smashed="yes">
+<attribute name="NAME" x="-150.495" y="876.935" size="1.27" layer="25"/>
+<attribute name="VALUE" x="-150.495" y="874.395" size="1.27" layer="27"/>
 </element>
 </elements>
@@
 <contactref element="Q10" pad="2"/>
 <contactref element="R125" pad="2"/>
+<contactref element="JP58" pad="3"/>
+<contactref element="JP59" pad="3"/>
 <wire x1="-134.62" y1="392.43" x2="-134.62" y2="384.81" width="0" layer="19" extent="1-1"/>
 <wire x1="-134.62" y1="372.11" x2="-134.62" y2="384.81" width="0" layer="19" extent="1-1"/>
@@
 <wire x1="-148.78" y1="831.85" x2="-148.78" y2="816.61" width="0" layer="19" extent="1-1"/>
 <wire x1="-147.94" y1="842.38" x2="-148.78" y2="831.85" width="0" layer="19" extent="1-1"/>
+<wire x1="-144.78" y1="857.25" x2="-147.94" y2="842.38" width="0" layer="19" extent="1-1"/>
+<wire x1="-144.78" y1="864.87" x2="-144.78" y2="857.25" width="0" layer="19" extent="1-1"/>
 <wire x1="-137.16" y1="205.22" x2="-134.62" y2="289.56" width="0" layer="19" extent="1-1"/>
 <wire x1="-137.16" y1="193.79" x2="-137.16" y2="205.22" width="0" layer="19" extent="1-1"/>
@@
 <contactref element="U1" pad="78"/>
 <contactref element="R119" pad="2"/>
-<wire x1="-85.17" y1="-949.9" x2="-140.12" y2="535.94" width="0" layer="19" extent="1-1"/>
+<contactref element="R130" pad="1"/>
+<wire x1="-140.12" y1="535.94" x2="-150.71" y2="876.3" width="0" layer="19" extent="1-1"/>
+<wire x1="-85.17" y1="-949.9" x2="-150.71" y2="876.3" width="0" layer="19" extent="1-1"/>
 </signal>
 <signal name="ESP_COM_RX">
 <contactref element="U1" pad="79"/>
 <contactref element="R118" pad="2"/>
-<wire x1="-85.67" y1="-949.9" x2="-140.12" y2="530.86" width="0" layer="19" extent="1-1"/>
+<contactref element="R129" pad="1"/>
+<wire x1="-140.12" y1="530.86" x2="-150.71" y2="871.22" width="0" layer="19" extent="1-1"/>
+<wire x1="-85.67" y1="-949.9" x2="-150.71" y2="871.22" width="0" layer="19" extent="1-1"/>
 </signal>
 <signal name="ESP_PROG_TX">
@@
 <contactref element="IM6" pad="35"/>
 <contactref element="R120" pad="1"/>
+<contactref element="R128" pad="1"/>
+<wire x1="-141.82" y1="541.02" x2="-150.71" y2="-1559.56" width="0" layer="19" extent="1-1"/>
 <wire x1="16.51" y1="39.624" x2="-141.82" y2="541.02" width="0" layer="19" extent="1-1"/>
 </signal>
@@
 <contactref element="IM6" pad="34"/>
 <contactref element="R121" pad="1"/>
+<contactref element="R127" pad="1"/>
+<wire x1="-141.82" y1="546.1" x2="-150.71" y2="-1554.48" width="0" layer="19" extent="1-1"/>
 <wire x1="19.05" y1="39.624" x2="-141.82" y2="546.1" width="0" layer="19" extent="1-1"/>
 </signal>
@@
 <wire x1="-150.71" y1="-1544.32" x2="-149.01" y2="-1549.4" width="0" layer="19" extent="1-1"/>
 </signal>
+<signal name="ESP-UART-RX">
+<contactref element="R127" pad="2"/>
+<contactref element="JP58" pad="1"/>
+<wire x1="-149.01" y1="-1554.48" x2="-149.86" y2="857.25" width="0" layer="19" extent="1-1"/>
+</signal>
+<signal name="ESP-UART-TX">
+<contactref element="R128" pad="2"/>
+<contactref element="JP58" pad="2"/>
+<wire x1="-149.01" y1="-1559.56" x2="-147.32" y2="857.25" width="0" layer="19" extent="1-1"/>
+</signal>
+<signal name="EXPANDER-UART-RX">
+<contactref element="R129" pad="2"/>
+<contactref element="JP59" pad="1"/>
+<wire x1="-149.86" y1="864.87" x2="-149.01" y2="871.22" width="0" layer="19" extent="1-1"/>
+</signal>
+<signal name="EXPANDER-UART-TX">
+<contactref element="R130" pad="2"/>
+<contactref element="JP59" pad="2"/>
+<wire x1="-147.32" y1="864.87" x2="-149.01" y2="876.3" width="0" layer="19" extent="1-1"/>
+</signal>
 </signals>

Commit message: MainBoardSCH: Add power connectors
Parts:
- added JP60: +3V3STM, pinhead:2X04
- added JP61: +3V3, pinhead:2X04
- added JP62: +5V, pinhead:2X04
- added JP63: VCC, pinhead:2X04
Connections:
- net +3V3: now also JP61.1, JP61.3, JP61.5, JP61.7
- net +3V3S: now also JP60.1, JP60.3, JP60.5, JP60.7
- net +5V: now also JP62.1, JP62.3, JP62.5, JP62.7
- net GND: now also JP60.2, JP60.4, JP60.6, JP60.8, JP61.2, JP61.4, JP61.6, JP61.8, JP62.2, JP62.4, JP62.6, JP62.8, JP63.2, JP63.4, JP63.6, JP63.8
- net VCC: now also JP63.1, JP63.3, JP63.5, JP63.7

Commit message: MainBoardSCH: Add ON_SW connector and OFF button
Parts:
- added BTN5: CHOOSE_ME, Switch:TL3342F160QG/TR
- added JP64: ON_SW, pinhead:1X02
- added R131: 180R, rcl_upravena:R0603
- JP23: device pinhead:2X04 -> pinhead:2X05
Connections:
- removed net !PWR_BTN: Q9.3
- removed net BUTTON0: U1.37
- new net BUTTON-OFF: BTN5.3, BTN5.4, JP23.9, R131.2
- net BAT+_PROTECTED: now also JP64.1
- net BUTTON1: now also U1.37
- net BUTTON_OFF: now also R131.1
- net BUTTON_ON: now also Q9.3
- net GND: now also BTN5.1, BTN5.2, JP23.10
- net PWR_BTN: now also JP64.2
Changed lines of the file:
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@@
 <attribute name="VALUE" x="-99.06" y="-1025.525" size="1.27" layer="27"/>
 </element>
-<element name="JP23" library="pinhead" library_urn="urn:adsk.eagle:library:325" package="2X04" package3d_urn="urn:adsk.eagle:package:22461/2" value="BUTTONS" x="-93.98" y="-1028.7" smashed="yes">
+<element name="JP23" library="pinhead" library_urn="urn:adsk.eagle:library:325" package="2X05" package3d_urn="urn:adsk.eagle:package:22470/2" value="BUTTONS" x="-93.98" y="-1028.7" smashed="yes">
 <attribute name="NAME" x="-99.06" y="-1025.525" size="1.27" layer="25" ratio="10"/>
-<attribute name="POPULARITY" value="47" x="-93.98" y="-1028.7" size="1.778" layer="27" display="off"/>
+<attribute name="POPULARITY" value="35" x="-93.98" y="-1028.7" size="1.778" layer="27" display="off"/>
 <attribute name="VALUE" x="-99.06" y="-1033.145" size="1.27" layer="27"/>
 </element>
@@
 <attribute name="VALUE" x="-152.4" y="899.795" size="1.27" layer="27"/>
 </element>
+<element name="R131" library="rcl_upravena" package="R0603" value="180R" x="-151.13" y="-1574.8" smashed="yes">
+<attribute name="NAME" x="-151.765" y="-1574.165" size="1.27" layer="25"/>
+<attribute name="VALUE" x="-151.765" y="-1576.705" size="1.27" layer="27"/>
+</element>
+<element name="BTN5" library="Switch" package="TL3342F160QG/TR" value="CHOOSE_ME" x="-160.02" y="-1570.99" smashed="yes">
+<attribute name="CREATED_BY" value="PCBLayout.com" x="-160.02" y="-1570.99" size="1.778" layer="27" display="off"/>
+<attribute name="DIGI_KEY_PART_NUMBER" value="EG2531CT-ND" x="-160.02" y="-1570.99" size="1.778" layer="27" display="off"/>
+<attribute name="MANUFACTURER" value="E-Switch" x="-160.02" y="-1570.99" size="1.778" layer="27" display="off"/>
+<attribute name="MPN" value="TL3342F160QG/TR" x="-160.02" y="-1570.99" size="1.778" layer="27" display="off"/>
+<attribute name="NAME" x="-163.83" y="-1567.18" size="1.778" layer="25"/>
+<attribute name="PACKAGE" value="SPST_NO" x="-160.02" y="-1570.99" size="1.778" layer="27" display="off"/>
+<attribute name="VALUE" x="-163.83" y="-1576.07" size="1.778" layer="27"/>
+</element>
+<element name="JP64" library="pinhead" library_urn="urn:adsk.eagle:library:325" package="1X02" package3d_urn="urn:adsk.eagle:package:22435/2" value="ON_SW" x="-162.56" y="-1581.15" smashed="yes">
+<attribute name="NAME" x="-163.9062" y="-1579.3212" size="1.27" layer="25" ratio="10"/>
+<attribute name="POPULARITY" value="98" x="-162.56" y="-1581.15" size="1.778" layer="27" display="off"/>
+<attribute name="VALUE" x="-163.83" y="-1584.325" size="1.27" layer="27"/>
+</element>
 </elements>
 <signals>
@@
 <contactref element="JP63" pad="6"/>
 <contactref element="JP63" pad="8"/>
+<contactref element="BTN5" pad="2"/>
+<contactref element="BTN5" pad="1"/>
+<contactref element="JP23" pad="10"/>
 <wire x1="-148.59" y1="905.51" x2="-146.05" y2="905.51" width="0" layer="19" extent="1-1"/>
 <wire x1="-151.13" y1="905.51" x2="-148.59" y2="905.51" width="0" layer="19" extent="1-1"/>
@@
 <wire x1="-98.54" y1="-1010.92" x2="-98.89" y2="-1005.84" width="0" layer="19" extent="1-1"/>
 <wire x1="-98.64" y1="-1016" x2="-98.54" y2="-1010.92" width="0" layer="19" extent="1-1"/>
-<wire x1="-97.79" y1="-1027.43" x2="-98.64" y2="-1016" width="0" layer="19" extent="1-1"/>
-<wire x1="-95.25" y1="-1027.43" x2="-97.79" y2="-1027.43" width="0" layer="19" extent="1-1"/>
-<wire x1="-92.71" y1="-1027.43" x2="-95.25" y2="-1027.43" width="0" layer="19" extent="1-1"/>
-<wire x1="-90.17" y1="-1027.43" x2="-92.71" y2="-1027.43" width="0" layer="19" extent="1-1"/>
-<wire x1="-90.17" y1="-1035.05" x2="-90.17" y2="-1027.43" width="0" layer="19" extent="1-1"/>
+<wire x1="-99.06" y1="-1027.43" x2="-98.64" y2="-1016" width="0" layer="19" extent="1-1"/>
+<wire x1="-96.52" y1="-1027.43" x2="-99.06" y2="-1027.43" width="0" layer="19" extent="1-1"/>
+<wire x1="-93.98" y1="-1027.43" x2="-96.52" y2="-1027.43" width="0" layer="19" extent="1-1"/>
+<wire x1="-91.44" y1="-1027.43" x2="-93.98" y2="-1027.43" width="0" layer="19" extent="1-1"/>
+<wire x1="-88.9" y1="-1027.43" x2="-91.44" y2="-1027.43" width="0" layer="19" extent="1-1"/>
+<wire x1="-90.17" y1="-1035.05" x2="-91.44" y2="-1027.43" width="0" layer="19" extent="1-1"/>
 <wire x1="-98.54" y1="-1038.86" x2="-90.17" y2="-1035.05" width="0" layer="19" extent="1-1"/>
 <wire x1="-98.54" y1="-1043.94" x2="-98.54" y2="-1038.86" width="0" layer="19" extent="1-1"/>
@@
 <wire x1="-144.78" y1="-1565.91" x2="-147.32" y2="-1565.91" width="0" layer="19" extent="1-1"/>
 <wire x1="-142.24" y1="-1565.91" x2="-144.78" y2="-1565.91" width="0" layer="19" extent="1-1"/>
+<wire x1="-156.87" y1="-1572.89" x2="-149.86" y2="-1565.91" width="0" layer="19" extent="1-1"/>
+<wire x1="-163.17" y1="-1572.89" x2="-156.87" y2="-1572.89" width="0" layer="19" extent="1-1"/>
 </signal>
 <signal name="+3V3">
@@
 <contactref element="SW_ON" pad="2"/>
 <contactref element="SW_ON" pad="1"/>
+<contactref element="JP64" pad="1"/>
 <wire x1="-50.19" y1="-448.94" x2="-56.49" y2="-448.94" width="0" layer="19" extent="1-1"/>
 <wire x1="65.573" y1="47.322" x2="-50.19" y2="-448.94" width="0" layer="19" extent="1-1"/>
@@
 <wire x1="66.873" y1="57.58" x2="66.223" y2="57.58" width="0" layer="19" extent="1-1"/>
 <wire x1="67.523" y1="57.58" x2="66.873" y2="57.58" width="0" layer="19" extent="1-1"/>
+<wire x1="-163.83" y1="-1581.15" x2="-56.49" y2="-448.94" width="0" layer="19" extent="1-1"/>
 </signal>
 <signal name="BAT+">
@@
 <contactref element="Q8" pad="1"/>
 <contactref element="R1" pad="2"/>
+<contactref element="JP64" pad="2"/>
 <wire x1="-50.19" y1="-445.14" x2="-56.49" y2="-445.14" width="0" layer="19" extent="1-1"/>
 <wire x1="-53.99" y1="-460.64" x2="-56.49" y2="-445.14" width="0" layer="19" extent="1-1"/>
 <wire x1="-53.99" y1="-468.26" x2="-53.99" y2="-460.64" width="0" layer="19" extent="1-1"/>
 <wire x1="-55.03" y1="-487.68" x2="-53.99" y2="-468.26" width="0" layer="19" extent="1-1"/>
-</signal>
-<signal name="!PWR_BTN">
-<contactref element="Q9" pad="3"/>
+<wire x1="-161.29" y1="-1581.15" x2="-56.49" y2="-445.14" width="0" layer="19" extent="1-1"/>
 </signal>
 <signal name="POWER">
@@
 <wire x1="-82.49" y1="-954.58" x2="-138.01" y2="-1201.42" width="0" layer="19" extent="1-1"/>
 </signal>
-<signal name="BUTTON0">
-<contactref element="U1" pad="37"/>
-</signal>
 <signal name="UTS1_TRIG">
 <contactref element="U1" pad="95"/>
@@
 <signal name="BUTTON_ON">
 <contactref element="U1" pad="7"/>
+<contactref element="Q9" pad="3"/>
+<wire x1="-53.34" y1="-466.46" x2="-97.85" y2="-954.58" width="0" layer="19" extent="1-1"/>
 </signal>
 <signal name="ESP_COM_TX">
@@
 <signal name="BUTTON_OFF">
 <contactref element="U1" pad="46"/>
+<contactref element="R131" pad="1"/>
+<wire x1="-86.17" y1="-965.26" x2="-151.98" y2="-1574.8" width="0" layer="19" extent="1-1"/>
 </signal>
 <signal name="N$1">
@@
 <signal name="BUTTON1">
 <contactref element="R34" pad="1"/>
+<contactref element="U1" pad="37"/>
+<wire x1="-90.67" y1="-965.26" x2="-132.93" y2="-1064.26" width="0" layer="19" extent="1-1"/>
 </signal>
 <signal name="BUTTON-1">
@@
 <contactref element="BTN1" pad="3"/>
 <contactref element="JP23" pad="1"/>
-<wire x1="-97.79" y1="-1029.97" x2="-131.23" y2="-1064.26" width="0" layer="19" extent="1-1"/>
+<wire x1="-99.06" y1="-1029.97" x2="-131.23" y2="-1064.26" width="0" layer="19" extent="1-1"/>
 <wire x1="-92.1" y1="174.62" x2="-131.23" y2="-1064.26" width="0" layer="19" extent="1-1"/>
 <wire x1="-98.4" y1="174.62" x2="-92.1" y2="174.62" width="0" layer="19" extent="1-1"/>
@@
 <wire x1="-109.83" y1="-1053.47" x2="-131.23" y2="-1069.34" width="0" layer="19" extent="1-1"/>
 <wire x1="-103.53" y1="-1053.47" x2="-109.83" y2="-1053.47" width="0" layer="19" extent="1-1"/>
-<wire x1="-95.25" y1="-1029.97" x2="-103.53" y2="-1053.47" width="0" layer="19" extent="1-1"/>
+<wire x1="-96.52" y1="-1029.97" x2="-103.53" y2="-1053.47" width="0" layer="19" extent="1-1"/>
 </signal>
 <signal name="BUTTON-3">
@@
 <wire x1="-121.26" y1="-1053.47" x2="-131.23" y2="-1074.42" width="0" layer="19" extent="1-1"/>
 <wire x1="-114.96" y1="-1053.47" x2="-121.26" y2="-1053.47" width="0" layer="19" extent="1-1"/>
-<wire x1="-92.71" y1="-1029.97" x2="-114.96" y2="-1053.47" width="0" layer="19" extent="1-1"/>
+<wire x1="-93.98" y1="-1029.97" x2="-114.96" y2="-1053.47" width="0" layer="19" extent="1-1"/>
 </signal>
 <signal name="BUTTON-4">
@@
 <wire x1="-132.69" y1="-1053.47" x2="-131.23" y2="-1079.5" width="0" layer="19" extent="1-1"/>
 <wire x1="-126.39" y1="-1053.47" x2="-132.69" y2="-1053.47" width="0" layer="19" extent="1-1"/>
-<wire x1="-90.17" y1="-1029.97" x2="-126.39" y2="-1053.47" width="0" layer="19" extent="1-1"/>
+<wire x1="-91.44" y1="-1029.97" x2="-126.39" y2="-1053.47" width="0" layer="19" extent="1-1"/>
 </signal>
 <signal name="LED_1">
@@
 <wire x1="-147.32" y1="864.87" x2="-149.01" y2="876.3" width="0" layer="19" extent="1-1"/>
 </signal>
+<signal name="BUTTON-OFF">
+<contactref element="R131" pad="2"/>
+<contactref element="BTN5" pad="4"/>
+<contactref element="BTN5" pad="3"/>
+<contactref element="JP23" pad="9"/>
+<wire x1="-156.87" y1="-1569.09" x2="-163.17" y2="-1569.09" width="0" layer="19" extent="1-1"/>
+<wire x1="-150.28" y1="-1574.8" x2="-156.87" y2="-1569.09" width="0" layer="19" extent="1-1"/>
+<wire x1="-88.9" y1="-1029.97" x2="-156.87" y2="-1569.09" width="0" layer="19" extent="1-1"/>
+</signal>
 </signals>

Commit message: MainBoardSCH: Add STM BOOT pins logic
Parts:
- added JP65: BOOT, pinhead:1X06
- added Q11: CHOOSE_ME, transistors:SOT323
- added R132, R133: 100k, rcl_upravena:R0603
Connections:
- new net BOOT1: JP65.4, R133.2
- new net BOOT1_PULL-DOWN: Q11.3, R133.1
- net +3V3S: now also JP65.1, JP65.3
- net BOOT0: now also JP65.2, Q11.1, R132.1
- net GND: now also JP65.6, Q11.2, R132.2
- net NRST: now also JP65.5
Changed lines of the file:
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@@
 <attribute name="VALUE" x="-163.83" y="-1584.325" size="1.27" layer="27"/>
+</element>
+<element name="JP65" library="pinhead" library_urn="urn:adsk.eagle:library:325" package="1X06" package3d_urn="urn:adsk.eagle:package:22472/2" value="BOOT" x="-157.48" y="913.13" smashed="yes">
+<attribute name="NAME" x="-165.1762" y="914.9588" size="1.27" layer="25" ratio="10"/>
+<attribute name="POPULARITY" value="79" x="-157.48" y="-1588.77" size="1.778" layer="27" display="off"/>
+<attribute name="VALUE" x="-165.1" y="909.955" size="1.27" layer="27"/>
+</element>
+<element name="R132" library="rcl_upravena" package="R0603" value="100k" x="-163.83" y="-1587.5" smashed="yes">
+<attribute name="NAME" x="-164.465" y="-1586.865" size="1.27" layer="25"/>
+<attribute name="VALUE" x="-164.465" y="-1589.405" size="1.27" layer="27"/>
+</element>
+<element name="Q11" library="transistors" package="SOT323" value="CHOOSE_ME" x="-163.83" y="-1593.85" smashed="yes">
+<attribute name="NAME" x="-165.735" y="-1592.345" size="1.27" layer="25"/>
+<attribute name="VALUE" x="-165.735" y="-1596.625" size="1.27" layer="27"/>
+</element>
+<element name="R133" library="rcl_upravena" package="R0603" value="100k" x="-163.83" y="-1600.2" smashed="yes">
+<attribute name="NAME" x="-164.465" y="-1599.565" size="1.27" layer="25"/>
+<attribute name="VALUE" x="-164.465" y="-1602.105" size="1.27" layer="27"/>
 </element>
 </elements>
@@
 <contactref element="BTN5" pad="1"/>
 <contactref element="JP23" pad="10"/>
+<contactref element="JP65" pad="6"/>
+<contactref element="R132" pad="2"/>
+<contactref element="Q11" pad="2"/>
 <wire x1="-148.59" y1="905.51" x2="-146.05" y2="905.51" width="0" layer="19" extent="1-1"/>
 <wire x1="-151.13" y1="905.51" x2="-148.59" y2="905.51" width="0" layer="19" extent="1-1"/>
 <wire x1="-143.51" y1="905.51" x2="-146.05" y2="905.51" width="0" layer="19" extent="1-1"/>
+<wire x1="-151.13" y1="913.13" x2="-151.13" y2="905.51" width="0" layer="19" extent="1-1"/>
 <wire x1="-143.51" y1="895.35" x2="-143.51" y2="905.51" width="0" layer="19" extent="1-1"/>
 <wire x1="-146.05" y1="895.35" x2="-143.51" y2="895.35" width="0" layer="19" extent="1-1"/>
@@
 <wire x1="-156.87" y1="-1572.89" x2="-149.86" y2="-1565.91" width="0" layer="19" extent="1-1"/>
 <wire x1="-163.17" y1="-1572.89" x2="-156.87" y2="-1572.89" width="0" layer="19" extent="1-1"/>
+<wire x1="-162.98" y1="-1587.5" x2="-163.17" y2="-1572.89" width="0" layer="19" extent="1-1"/>
+<wire x1="-163.18" y1="-1594.75" x2="-162.98" y2="-1587.5" width="0" layer="19" extent="1-1"/>
 </signal>
 <signal name="+3V3">
@@
 <contactref element="JP60" pad="3"/>
 <contactref element="JP60" pad="5"/>
+<contactref element="JP65" pad="1"/>
+<contactref element="JP65" pad="3"/>
 <wire x1="-65.09" y1="-690.71" x2="-65.09" y2="-698.33" width="0" layer="19" extent="1-1"/>
 <wire x1="-65.09" y1="-683.09" x2="-65.09" y2="-690.71" width="0" layer="19" extent="1-1"/>
@@
 <wire x1="-140.22" y1="659.13" x2="-137.414" y2="246.38" width="0" layer="19" extent="1-1"/>
 <wire x1="-143.255" y1="709.93" x2="-140.22" y2="659.13" width="0" layer="19" extent="1-1"/>
+<wire x1="-158.75" y1="913.13" x2="-143.255" y2="709.93" width="0" layer="19" extent="1-1"/>
+<wire x1="-163.83" y1="913.13" x2="-158.75" y2="913.13" width="0" layer="19" extent="1-1"/>
 </signal>
 <signal name="PWRLED_VCC">
@@
 <signal name="BOOT0">
 <contactref element="U1" pad="94"/>
+<contactref element="JP65" pad="2"/>
+<contactref element="R132" pad="1"/>
+<contactref element="Q11" pad="1"/>
+<wire x1="-164.48" y1="-1594.75" x2="-161.29" y2="913.13" width="0" layer="19" extent="1-1"/>
+<wire x1="-164.68" y1="-1587.5" x2="-164.48" y2="-1594.75" width="0" layer="19" extent="1-1"/>
+<wire x1="-93.17" y1="-949.9" x2="-164.68" y2="-1587.5" width="0" layer="19" extent="1-1"/>
 </signal>
 <signal name="NRST">
 <contactref element="U1" pad="14"/>
 <contactref element="R71" pad="1"/>
+<contactref element="JP65" pad="5"/>
+<wire x1="-97.85" y1="-958.08" x2="-153.67" y2="913.13" width="0" layer="19" extent="1-1"/>
 <wire x1="-138.01" y1="-1145.54" x2="-97.85" y2="-958.08" width="0" layer="19" extent="1-1"/>
 </signal>
@@
 <wire x1="-88.9" y1="-1029.97" x2="-156.87" y2="-1569.09" width="0" layer="19" extent="1-1"/>
 </signal>
+<signal name="BOOT1">
+<contactref element="JP65" pad="4"/>
+<contactref element="R133" pad="2"/>
+<wire x1="-162.98" y1="-1600.2" x2="-156.21" y2="913.13" width="0" layer="19" extent="1-1"/>
+</signal>
+<signal name="BOOT1_PULL-DOWN">
+<contactref element="R133" pad="1"/>
+<contactref element="Q11" pad="3"/>
+<wire x1="-163.83" y1="-1592.95" x2="-164.68" y2="-1600.2" width="0" layer="19" extent="1-1"/>
+</signal>
 </signals>
