File: ele/MainBoard/RBCX-MainBoard.sch (EAGLE design)
At the start: 311 parts, among them IC1 AMS1117-3.3, IC10 INA180A4, IC11 INA180A4, IC2 DRV8833PWP, IC3 INA180A4, IC4 INA180A4, IC5 DRV8833PWP, IC6 INA180A4, IC7 INA180A4, IC8 INA180A4, IC9 INA180A4, Q1 NCE20P45Q, Q10 CHOOSE_ME, Q11 CHOOSE_ME, Q2 NCE20P45Q, Q3 CHOOSE_ME, Q4 CHOOSE_ME, Q5 CHOOSE_ME, Q6 CHOOSE_ME, Q7 CHOOSE_ME, Q8 CHOOSE_ME, Q9 CHOOSE_ME, SW1 CHOOSE_ME, SW2 CHOOSE_ME, SW3 CHOOSE_ME, SW4 CHOOSE_ME, SW5 CHOOSE_ME, SW6 CHOOSE_ME, U1 STM32F103VCT6, X1 POWER_OUT, X10 52745-3090, X11 52745-2090, X2 POWER_IN, Y1 5032/2P, Y2 3215_2P

Commit message: MainBoardSCH: Add N channel MOSFETs type
Parts:
- Q10, Q11, Q3, Q4, Q5, Q6, Q7, Q8, Q9: value CHOOSE_ME -> 2N7002; device transistors:N-MOSFET-SOT323-GSD -> transistors:N-MOSFET-SOT23-GSD; DESCRIPTION (none) -> N MOSFET 60V 115mA 7Ω; EXTENDED (none) -> NO; LCSC_ID (none) -> C8545; MF (none) -> Changjiang Electronics Tech (CJ); MF_ID (none) -> 2N7002; PACKAGE (none) -> SOT-23-3; PADS (none) -> 3; PRICE_1PLUS (none) -> $0.0236; PRICE_200PLUS (none) -> $0.0113

Commit message: MainBoardSCH: Add missing P channel MOSFETs attributes (PADS, EXTENDED, MF)
Parts:
- Q1, Q2: EXTENDED (none) -> YES; MF (none) -> Wuxi NCE Power Semiconductor; PADS (none) -> 8
Changed lines of the file:
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@@
 <part name="Q1" library="transistors" deviceset="P-MOSFET" device="-MLP_HS" value="NCE20P45Q">
 <attribute name="DESCRIPTION" value="P MOSFET 19V 35A 7mΩ"/>
+<attribute name="EXTENDED" value="YES"/>
 <attribute name="LCSC_ID" value="C193354"/>
+<attribute name="MF" value="Wuxi NCE Power Semiconductor"/>
 <attribute name="MF_ID" value="NCE20P45Q"/>
 <attribute name="PACKAGE" value="DFN-8_EP_3.3x3.3x0.65P"/>
+<attribute name="PADS" value="8"/>
 <attribute name="PRICE_1000PLUS" value="$0.1218"/>
 <attribute name="PRICE_100PLUS" value="$0.1276"/>
@@
 <part name="Q2" library="transistors" deviceset="P-MOSFET" device="-MLP_HS" value="NCE20P45Q">
 <attribute name="DESCRIPTION" value="P MOSFET 19V 35A 7mΩ"/>
+<attribute name="EXTENDED" value="YES"/>
 <attribute name="LCSC_ID" value="C193354"/>
+<attribute name="MF" value="Wuxi NCE Power Semiconductor"/>
 <attribute name="MF_ID" value="NCE20P45Q"/>
 <attribute name="PACKAGE" value="DFN-8_EP_3.3x3.3x0.65P"/>
+<attribute name="PADS" value="8"/>
 <attribute name="PRICE_1000PLUS" value="$0.1218"/>
 <attribute name="PRICE_100PLUS" value="$0.1276"/>
@@
 <attribute name="PRICE_30PLUS" x="73.66" y="172.72" size="1.27" layer="96" rot="MR90" display="off"/>
 <attribute name="PRICE_500PLUS" x="73.66" y="172.72" size="1.27" layer="96" rot="MR90" display="off"/>
+<attribute name="EXTENDED" x="73.66" y="172.72" size="1.27" layer="96" rot="MR90" display="off"/>
+<attribute name="MF" x="73.66" y="172.72" size="1.27" layer="96" rot="MR90" display="off"/>
+<attribute name="PADS" x="73.66" y="172.72" size="1.27" layer="96" rot="MR90" display="off"/>
 </instance>
 <instance part="SW1" gate="1" x="83.82" y="157.48" smashed="yes" rot="MR180">
@@
 <attribute name="PRICE_30PLUS" x="109.22" y="172.72" size="1.27" layer="96" rot="R90" display="off"/>
 <attribute name="PRICE_500PLUS" x="109.22" y="172.72" size="1.27" layer="96" rot="R90" display="off"/>
+<attribute name="EXTENDED" x="109.22" y="172.72" size="1.27" layer="96" rot="R90" display="off"/>
+<attribute name="MF" x="109.22" y="172.72" size="1.27" layer="96" rot="R90" display="off"/>
+<attribute name="PADS" x="109.22" y="172.72" size="1.27" layer="96" rot="R90" display="off"/>
 </instance>
 <instance part="R66" gate="G$1" x="106.68" y="157.48" smashed="yes" rot="R90">

Commit message: MainBoard: Change resistors package to 0402, because of space and price
Parts:
- R1, R10, R100, R101, R102, R103, R104, R105, R106, R107, R108, R109, R11, R110, R111, R112, R113, R114, R115, R116, R117, R118, R119, R12, R120, R121, R122, R123, R124, R125, R126, R127, R128, R129, R13, R131, R132, R133, R134, R14, R15, R16, R17, R2, R20, R21, R22, R23, R24, R25, R3, R32, R34, R36, R38, R4, R40, R41, R42, R43, R45, R46, R47, R48, R49, R5, R50, R51, R52, R53, R54, R55, R56, R57, R58, R59, R6, R60, R61, R62, R63, R64, R65, R67, R68, R69, R7, R75, R76, R77, R78, R79, R8, R80, R81, R83, R87, R88, R9, R93: device rcl_upravena:R-EU_R0603 -> rcl_upravena:R-EU_R0402
