File: hw/RBCX_v1.3/Power.kicad_sch (KiCad schematic)
At the start: 82 parts

Commit message: Remove stepdowns, Micro-USB; fixup region names
Parts:
- removed IM1: (no value), symbol RBCX-eagle-import:STEPDOWN
- removed JP1: (no value), symbol RBCX-eagle-import:PINHD-1X1
- BAT1: value (none) -> CR2032; footprint (none) -> RBCX:SMD-BAT-CR2032-BS-6-1
- C1, C2: footprint (none) -> RBCX:E5-10,5
- C3, C4: footprint (none) -> RBCX:C0805
- C5, C7: footprint (none) -> RBCX:C0402
- C6, C8: footprint (none) -> RBCX:C0603
- D1: footprint (none) -> RBCX:SOD123
- D2, D3, D4, D5, D6, D7, D8: value (none) -> SS34; footprint (none) -> RBCX:SMA
- D9: value (none) -> BAS40-04; footprint (none) -> RBCX:SOT23
- IC1: value (none) -> AMS1117-3.3; footprint (none) -> RBCX:SOT223
- JP2: value (none) -> +3V3STM; footprint (none) -> RBCX:2X04
- JP3: value (none) -> +3V3; footprint (none) -> RBCX:2X04
- JP4: value (none) -> +5V; footprint (none) -> RBCX:2X04
- JP5: value (none) -> VCC; footprint (none) -> RBCX:2X04
- LED1, LED10, LED11, LED12, LED2, LED3, LED4, LED5, LED6, LED7, LED8, LED9: value (none) -> red; footprint (none) -> RBCX:CHIPLED_0603
- Q1, Q2: footprint (none) -> RBCX:MLP3.3X3.3_HS
- Q3, Q4: footprint (none) -> RBCX:SOT23
- R1: value (none) -> 100k; footprint (none) -> RBCX:R0402
- R10, R11, R2, R4, R6: value (none) -> 10k; footprint (none) -> RBCX:R0402
- R12, R13: value (none) -> 4k7; footprint (none) -> RBCX:R0402
- R14, R15, R20, R21, R22, R23: value (none) -> 2k2; footprint (none) -> RBCX:R0402
- R16, R17, R18, R19: value (none) -> 1k; footprint (none) -> RBCX:R0402
- R3, R8: value (none) -> 24k; footprint (none) -> RBCX:R0402
- R5: value (none) -> 330R; footprint (none) -> RBCX:R0402
- R7: value (none) -> 1M; footprint (none) -> RBCX:R0402
- R9: value (none) -> 5k6; footprint (none) -> RBCX:R0402
- S1, S2: value (none) -> TS-1187A-C-C-B; footprint (none) -> RBCX:TS-1187A
- TP1, TP10, TP12, TP13, TP14, TP2, TP3, TP4, TP5, TP6, TP7, TP8, TP9: value (none) -> TP_06MM; footprint (none) -> RBCX:TP_06
- TP11: value (none) -> TP_08MM; footprint (none) -> RBCX:TP_08
- X1: value (none) -> POWER_IN; footprint (none) -> RBCX:W237-133
- X2: value (none) -> POWER_OUT; footprint (none) -> RBCX:W237-132
Connections:
- net +5V: no longer D5.C, D6.A
