File: hw/RBCX_v1.3/PD.kicad_sch (KiCad schematic)
At the start: 27 parts

Commit message: Work in progress
Parts:
- removed LED? (x3): red, LED_SMD:LED_0603_1608Metric, symbol RBCX-eagle-import:LEDCHIPLED_0603
- removed Q? (x2): JSM3622, RBCX:JSM3622, symbol RBCX:JSM3622
- removed R?: 1k, Resistor_SMD:R_0201_0603Metric, symbol Device:R
- added D41, D42, D43, D44: red, LED_SMD:LED_0603_1608Metric, symbol Device:LED
- added R175: 4k7, Resistor_SMD:R_0201_0603Metric, symbol Device:R
- U22: renamed from U?; footprint (none) -> Package_DFN_QFN:QFN-24-1EP_4x4mm_P0.5mm_EP2.65x2.65mm
- gave numbers to parts that had none: 20
Connections:
- net GND: now also R175.1
- net USB_DM: no longer J49.3 (Pin_3), R179.2, U21.A6 (DP1), U21.B6 (DP2)
- net VUSB: now also C79.2, R172.2, U22.24 (VCC)
- net V_USB: now also D41.2 (A), D42.2 (A)
- net at U22.6 (GPIO4): now also D43.2 (A), D44.2 (A)
- net at R178.2: now also D43.1 (K)
- net at R174.2: now also D42.1 (K)
- net at R173.2: now also D41.1 (K)
- new net: D44.1 (K), R175.2
- new net USB_DP: J49.3 (Pin_3), R179.2, U21.A6 (DP1), U21.B6 (DP2)
- no-connect marks 2 -> 3
Other:
- moved on the sheet: C78
