File: hw/RBCX_v1.3/STM_connecors.kicad_sch (KiCad schematic)
At the start: 19 parts

Commit message: Work in progress
Parts:
- removed J?: Conn_02x04_Counter_Clockwise, Connector_PinHeader_2.54mm:PinHeader_2x04_P2.54mm_Vertical, symbol Connector_Generic:Conn_02x04_Counter_Clockwise
- added J42: Conn_02x04_Odd_Even, Connector_PinHeader_2.54mm:PinHeader_2x04_P2.54mm_Vertical, symbol Connector_Generic:Conn_02x04_Odd_Even
- gave numbers to parts that had none: 18
Connections:
- net 3V3: now also J42.5 (Pin_5), J42.6 (Pin_6)
- net 5V: now also J42.7 (Pin_7), J42.8 (Pin_8)
- net GND: now also J42.3 (Pin_3), J42.4 (Pin_4)
- net at R124.2: now also J42.1 (Pin_1)
- net at R125.1: now also J42.2 (Pin_2)
Other:
- moved on the sheet: J44, JP9, R124, R125, R128, R129

Commit message: New PCB layout
some changes of schema:
- change PD sink AO33772 to AO33771
- remove power switch
Parts:
- J41, J43, J44, J45, J46: footprint Connector_PinHeader_2.54mm:PinHeader_1x04_P2.54mm_Vertical -> RBCX:PinHeader_1x04_P2.54mm_Vertical
- J42: footprint Connector_PinHeader_2.54mm:PinHeader_2x04_P2.54mm_Vertical -> RBCX:PinHeader_2x04_P2.54mm_Vertical
Changed lines of the file:
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@@
       (effects (font (size 1.27 1.27)) (justify left))
     )
-    (property "Footprint" "Connector_PinHeader_2.54mm:PinHeader_1x04_P2.54mm_Vertical" (id 2) (at 68.58 64.77 0)
+    (property "Footprint" "RBCX:PinHeader_1x04_P2.54mm_Vertical" (id 2) (at 68.58 64.77 0)
       (effects (font (size 1.27 1.27)) hide)
     )
@@
       (effects (font (size 1.27 1.27)) (justify left))
     )
-    (property "Footprint" "Connector_PinHeader_2.54mm:PinHeader_1x04_P2.54mm_Vertical" (id 2) (at 125.73 69.85 0)
+    (property "Footprint" "RBCX:PinHeader_1x04_P2.54mm_Vertical" (id 2) (at 125.73 69.85 0)
       (effects (font (size 1.27 1.27)) hide)
     )
@@
       (effects (font (size 1.27 1.27)) (justify left))
     )
-    (property "Footprint" "Connector_PinHeader_2.54mm:PinHeader_1x04_P2.54mm_Vertical" (id 2) (at 68.58 36.83 0)
+    (property "Footprint" "RBCX:PinHeader_1x04_P2.54mm_Vertical" (id 2) (at 68.58 36.83 0)
       (effects (font (size 1.27 1.27)) hide)
     )
@@
       (effects (font (size 1.27 1.27)) (justify left))
     )
-    (property "Footprint" "Connector_PinHeader_2.54mm:PinHeader_1x04_P2.54mm_Vertical" (id 2) (at 68.58 92.71 0)
+    (property "Footprint" "RBCX:PinHeader_1x04_P2.54mm_Vertical" (id 2) (at 68.58 92.71 0)
       (effects (font (size 1.27 1.27)) hide)
     )
@@
     (property "Reference" "J42" (id 0) (at 163.83 43.18 0))
     (property "Value" "Conn_02x04_Odd_Even" (id 1) (at 163.83 45.72 0))
-    (property "Footprint" "Connector_PinHeader_2.54mm:PinHeader_2x04_P2.54mm_Vertical" (id 2) (at 162.56 52.07 0)
+    (property "Footprint" "RBCX:PinHeader_2x04_P2.54mm_Vertical" (id 2) (at 162.56 52.07 0)
       (effects (font (size 1.27 1.27)) hide)
     )
@@
       (effects (font (size 1.27 1.27)) (justify left))
     )
-    (property "Footprint" "Connector_PinHeader_2.54mm:PinHeader_1x04_P2.54mm_Vertical" (id 2) (at 68.58 120.65 0)
-      (effects (font (size 1.27 1.27)) hide)
-    )
+    (property "Footprint" "RBCX:PinHeader_1x04_P2.54mm_Vertical" (id 2) (at 68.58 120.65 0)
+      (effects (font (size 1.27 1.27)) hide)
+    )

Commit message: Production files
Parts:
- J41, J43, J44, J45, J46: JLCPCB_CORRECTION (none) -> 0;-3.81;90
- J42: JLCPCB_CORRECTION (none) -> 1.27;-3.81;90; LCSC C225289 -> C124386
Changed lines of the file:
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@@
+      (effects (font (size 1.27 1.27)) hide)
+    )
+    (property "JLCPCB_CORRECTION" "0;-3.81;90" (id 6) (at 68.58 64.77 0)
       (effects (font (size 1.27 1.27)) hide)
     )
@@
     )
     (property "Basic/Extended" "E" (id 5) (at 125.73 69.85 0)
+      (effects (font (size 1.27 1.27)) hide)
+    )
+    (property "JLCPCB_CORRECTION" "0;-3.81;90" (id 6) (at 125.73 69.85 0)
       (effects (font (size 1.27 1.27)) hide)
     )
@@
       (effects (font (size 1.27 1.27)) hide)
     )
+    (property "JLCPCB_CORRECTION" "0;-3.81;90" (id 6) (at 68.58 36.83 0)
+      (effects (font (size 1.27 1.27)) hide)
+    )
     (pin "1")
     (pin "2")
@@
     )
     (property "Basic/Extended" "E" (id 5) (at 68.58 92.71 0)
+      (effects (font (size 1.27 1.27)) hide)
+    )
+    (property "JLCPCB_CORRECTION" "0;-3.81;90" (id 6) (at 68.58 92.71 0)
       (effects (font (size 1.27 1.27)) hide)
     )
@@
       (effects (font (size 1.27 1.27)) hide)
     )
-    (property "LCSC" "C225289" (id 4) (at 162.56 52.07 0)
+    (property "LCSC" "C124386" (id 4) (at 162.56 52.07 0)
       (effects (font (size 1.27 1.27)) hide)
     )
     (property "Basic/Extended" "E" (id 5) (at 162.56 52.07 0)
+      (effects (font (size 1.27 1.27)) hide)
+    )
+    (property "JLCPCB_CORRECTION" "1.27;-3.81;90" (id 6) (at 162.56 52.07 0)
       (effects (font (size 1.27 1.27)) hide)
     )
@@
       (effects (font (size 1.27 1.27)) hide)
     )
+    (property "JLCPCB_CORRECTION" "0;-3.81;90" (id 6) (at 68.58 120.65 0)
+      (effects (font (size 1.27 1.27)) hide)
+    )
