File: hw/RBCX_v1.3/User_interface.kicad_sch (KiCad schematic)
At the start: 62 parts, among them J29 Conn_01x01, J30 Conn_02x04_Odd_Even, J31 Conn_02x04_Odd_Even, J32 Conn_01x02, J33 Conn_02x04_Odd_Even, Q5 Q_NMOS_DGS, Q6 Q_NMOS_DGS, SW1 SW, SW10 SW, SW11 SW, SW12 SW, SW2 SW, SW3 SW, SW4 SW, SW5 SW, SW6 SW, SW7 SW, SW8 SW, SW9 SW, U3 BAT54C, X2 52559-3092

Commit message: Production files
Parts:
- IM1, IM2, J29, TP11, X2: JLCPCB_IGNORE (none) -> 1
- J30, J31, J33: JLCPCB_CORRECTION (none) -> 1.27;-3.81;90; LCSC C225289 -> C124386
- Q5, Q6, U3: JLCPCB_CORRECTION (none) -> 0;0;180
Changed lines of the file:
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@@
+      (effects (font (size 1.27 1.27)) hide)
+    )
+    (property "JLCPCB_IGNORE" "1" (id 4) (at 269.24 88.9 0)
       (effects (font (size 1.27 1.27)) hide)
     )
@@
     )
     (property "Datasheet" "" (id 3) (at 269.24 43.18 0)
+      (effects (font (size 1.27 1.27)) hide)
+    )
+    (property "JLCPCB_IGNORE" "1" (id 4) (at 269.24 43.18 0)
       (effects (font (size 1.27 1.27)) hide)
     )
@@
       (effects (font (size 1.27 1.27)) hide)
     )
+    (property "JLCPCB_IGNORE" "1" (id 4) (at 269.24 58.42 0)
+      (effects (font (size 1.27 1.27)) hide)
+    )
     (pin "1")
     (pin "2")
@@
     )
     (property "Datasheet" "~" (id 3) (at 109.22 38.1 0)
+      (effects (font (size 1.27 1.27)) hide)
+    )
+    (property "JLCPCB_IGNORE" "1" (id 4) (at 109.22 38.1 0)
       (effects (font (size 1.27 1.27)) hide)
     )
@@
       (effects (font (size 1.27 1.27)) hide)
     )
+    (property "JLCPCB_IGNORE" "1" (id 4) (at 269.24 83.82 0)
+      (effects (font (size 1.27 1.27)) hide)
+    )
     (pin "1")
     (pin "2")
@@
     )
     (property "Datasheet" "" (id 3) (at 269.24 55.88 0)
+      (effects (font (size 1.27 1.27)) hide)
+    )
+    (property "JLCPCB_IGNORE" "1" (id 4) (at 269.24 55.88 0)
       (effects (font (size 1.27 1.27)) hide)
     )
@@
       (effects (font (size 1.27 1.27)) hide)
     )
+    (property "JLCPCB_IGNORE" "1" (id 4) (at 269.24 60.96 0)
+      (effects (font (size 1.27 1.27)) hide)
+    )
     (pin "1")
     (pin "2")
@@
     )
     (property "Datasheet" "" (id 3) (at 269.24 78.74 0)
+      (effects (font (size 1.27 1.27)) hide)
+    )
+    (property "JLCPCB_IGNORE" "1" (id 4) (at 269.24 78.74 0)
       (effects (font (size 1.27 1.27)) hide)
     )
@@
       (effects (font (size 1.27 1.27)) hide)
     )
-    (property "LCSC" "C225289" (id 4) (at 207.01 144.78 0)
+    (property "LCSC" "C124386" (id 4) (at 207.01 144.78 0)
       (effects (font (size 1.27 1.27)) hide)
     )
     (property "Basic/Extended" "E" (id 5) (at 207.01 144.78 0)
+      (effects (font (size 1.27 1.27)) hide)
+    )
+    (property "JLCPCB_CORRECTION" "1.27;-3.81;90" (id 6) (at 207.01 144.78 0)
       (effects (font (size 1.27 1.27)) hide)
     )
@@
       (effects (font (size 1.27 1.27)) hide)
     )
+    (property "JLCPCB_IGNORE" "1" (id 4) (at 269.24 35.56 0)
+      (effects (font (size 1.27 1.27)) hide)
+    )
     (pin "1")
     (pin "2")
@@
       (effects (font (size 1.27 1.27)) hide)
     )
+    (property "JLCPCB_CORRECTION" "0;0;180" (id 6) (at 248.92 148.59 0)
+      (effects (font (size 1.27 1.27)) hide)
+    )
     (pin "1")
     (pin "2")
@@
     )
     (property "Datasheet" "" (id 3) (at 269.24 76.2 0)
+      (effects (font (size 1.27 1.27)) hide)
+    )
+    (property "JLCPCB_IGNORE" "1" (id 4) (at 269.24 76.2 0)
       (effects (font (size 1.27 1.27)) hide)
     )
@@
       (effects (font (size 1.27 1.27)) hide)
     )
+    (property "JLCPCB_IGNORE" "1" (id 4) (at 269.24 40.64 0)
+      (effects (font (size 1.27 1.27)) hide)
+    )
     (pin "1")
     (pin "2")
@@
       (effects (font (size 1.27 1.27)) hide)
     )
+    (property "JLCPCB_IGNORE" "1" (id 4) (at 269.24 73.66 0)
+      (effects (font (size 1.27 1.27)) hide)
+    )
     (pin "1")
     (pin "2")
@@
     (in_bom yes) (on_board yes)
     (property "Reference" "IM2" (id 0) (at 68.58 165.1 0)
-      (effects (font (size 1.778 1.5113)) (justify left bottom))
+      (effects (font (size 1.778 1.5113)) (justify right bottom))
     )
     (property "Value" "DISPLAY-OLED-128X32" (id 1) (at 68.58 168.91 0)
@@
       (effects (font (size 1.27 1.27)) hide)
     )
+    (property "JLCPCB_IGNORE" "1" (id 4) (at 88.9 176.53 0)
+      (effects (font (size 1.27 1.27)) hide)
+    )
     (pin "1")
     (pin "2")
@@
     )
     (property "Datasheet" "" (id 3) (at 269.24 38.1 0)
+      (effects (font (size 1.27 1.27)) hide)
+    )
+    (property "JLCPCB_IGNORE" "1" (id 4) (at 269.24 38.1 0)
       (effects (font (size 1.27 1.27)) hide)
     )
@@
       (effects (font (size 1.27 1.27)) hide)
     )
-    (property "LCSC" "C225289" (id 4) (at 207.01 127 0)
+    (property "LCSC" "C124386" (id 4) (at 207.01 127 0)
       (effects (font (size 1.27 1.27)) hide)
     )
     (property "Basic/Extended" "E" (id 5) (at 207.01 127 0)
+      (effects (font (size 1.27 1.27)) hide)
+    )
+    (property "JLCPCB_CORRECTION" "1.27;-3.81;90" (id 6) (at 207.01 127 0)
       (effects (font (size 1.27 1.27)) hide)
     )
@@
       (effects (font (size 1.27 1.27)) hide)
     )
+    (property "JLCPCB_IGNORE" "1" (id 4) (at 269.24 109.22 0)
+      (effects (font (size 1.27 1.27)) hide)
+    )
     (pin "1")
     (pin "2")
@@
       (effects (font (size 1.27 1.27)) hide)
     )
+    (property "JLCPCB_IGNORE" "1" (id 4) (at 256.54 127 0)
+      (effects (font (size 1.27 1.27)) hide)
+    )
     (pin "P$1")
   )
@@
     )
     (property "Datasheet" "" (id 3) (at 269.24 86.36 0)
+      (effects (font (size 1.27 1.27)) hide)
+    )
+    (property "JLCPCB_IGNORE" "1" (id 4) (at 269.24 86.36 0)
       (effects (font (size 1.27 1.27)) hide)
     )
@@
       (effects (font (size 1.27 1.27)) hide)
     )
-    (property "LCSC" "C225289" (id 4) (at 69.85 97.79 0)
+    (property "LCSC" "C124386" (id 4) (at 69.85 97.79 0)
       (effects (font (size 1.27 1.27)) hide)
     )
     (property "Basic/Extended" "E" (id 5) (at 69.85 97.79 0)
+      (effects (font (size 1.27 1.27)) hide)
+    )
+    (property "JLCPCB_CORRECTION" "1.27;-3.81;90" (id 6) (at 69.85 97.79 0)
       (effects (font (size 1.27 1.27)) hide)
     )
@@
       (effects (font (size 1.27 1.27)) hide)
     )
+    (property "JLCPCB_IGNORE" "1" (id 4) (at 269.24 63.5 0)
+      (effects (font (size 1.27 1.27)) hide)
+    )
     (pin "1")
     (pin "2")
@@
     )
     (property "Datasheet" "" (id 3) (at 269.24 93.98 0)
+      (effects (font (size 1.27 1.27)) hide)
+    )
+    (property "JLCPCB_IGNORE" "1" (id 4) (at 269.24 93.98 0)
       (effects (font (size 1.27 1.27)) hide)
     )
@@
     )
     (property "Datasheet" "" (id 3) (at 52.07 151.003 0)
+      (effects (font (size 1.27 1.27)) hide)
+    )
+    (property "JLCPCB_IGNORE" "1" (id 4) (at 52.07 151.003 0)
       (effects (font (size 1.27 1.27)) hide)
     )
@@
       (effects (font (size 1.27 1.27)) hide)
     )
+    (property "JLCPCB_IGNORE" "1" (id 4) (at 269.24 104.14 0)
+      (effects (font (size 1.27 1.27)) hide)
+    )
     (pin "1")
     (pin "2")
@@
       (effects (font (size 1.27 1.27)) hide)
     )
+    (property "JLCPCB_IGNORE" "1" (id 4) (at 269.24 106.68 0)
+      (effects (font (size 1.27 1.27)) hide)
+    )
     (pin "1")
     (pin "2")
@@
     )
     (property "Datasheet" "" (id 3) (at 269.24 96.52 0)
+      (effects (font (size 1.27 1.27)) hide)
+    )
+    (property "JLCPCB_IGNORE" "1" (id 4) (at 269.24 96.52 0)
       (effects (font (size 1.27 1.27)) hide)
     )
@@
       (effects (font (size 1.27 1.27)) hide)
     )
+    (property "JLCPCB_IGNORE" "1" (id 4) (at 269.24 68.58 0)
+      (effects (font (size 1.27 1.27)) hide)
+    )
     (pin "1")
     (pin "2")
@@
     )
     (property "Datasheet" "" (id 3) (at 269.24 71.12 0)
+      (effects (font (size 1.27 1.27)) hide)
+    )
+    (property "JLCPCB_IGNORE" "1" (id 4) (at 269.24 71.12 0)
       (effects (font (size 1.27 1.27)) hide)
     )
@@
       (effects (font (size 1.27 1.27)) hide)
     )
+    (property "JLCPCB_CORRECTION" "0;0;180" (id 6) (at 165.1 127 0)
+      (effects (font (size 1.27 1.27)) hide)
+    )
     (pin "1")
     (pin "2")
@@
     )
     (property "Datasheet" "" (id 3) (at 269.24 66.04 0)
+      (effects (font (size 1.27 1.27)) hide)
+    )
+    (property "JLCPCB_IGNORE" "1" (id 4) (at 269.24 66.04 0)
       (effects (font (size 1.27 1.27)) hide)
     )
@@
     )
     (property "Datasheet" "" (id 3) (at 269.24 48.26 0)
+      (effects (font (size 1.27 1.27)) hide)
+    )
+    (property "JLCPCB_IGNORE" "1" (id 4) (at 269.24 48.26 0)
       (effects (font (size 1.27 1.27)) hide)
     )
@@
       (effects (font (size 1.27 1.27)) hide)
     )
+    (property "JLCPCB_IGNORE" "1" (id 4) (at 269.24 45.72 0)
+      (effects (font (size 1.27 1.27)) hide)
+    )
     (pin "1")
     (pin "2")
@@
       (effects (font (size 1.27 1.27)) hide)
     )
+    (property "JLCPCB_IGNORE" "1" (id 4) (at 269.24 50.8 0)
+      (effects (font (size 1.27 1.27)) hide)
+    )
     (pin "1")
     (pin "2")
@@
     )
     (property "Datasheet" "" (id 3) (at 269.24 101.6 0)
+      (effects (font (size 1.27 1.27)) hide)
+    )
+    (property "JLCPCB_IGNORE" "1" (id 4) (at 269.24 101.6 0)
       (effects (font (size 1.27 1.27)) hide)
     )
@@
     )
     (property "Datasheet" "" (id 3) (at 269.24 81.28 0)
+      (effects (font (size 1.27 1.27)) hide)
+    )
+    (property "JLCPCB_IGNORE" "1" (id 4) (at 269.24 81.28 0)
       (effects (font (size 1.27 1.27)) hide)
     )
@@
       (effects (font (size 1.27 1.27)) hide)
     )
+    (property "JLCPCB_IGNORE" "1" (id 4) (at 269.24 53.34 0)
+      (effects (font (size 1.27 1.27)) hide)
+    )
     (pin "1")
     (pin "2")
@@
     )
     (property "Datasheet" "" (id 3) (at 269.24 99.06 0)
+      (effects (font (size 1.27 1.27)) hide)
+    )
+    (property "JLCPCB_IGNORE" "1" (id 4) (at 269.24 99.06 0)
       (effects (font (size 1.27 1.27)) hide)
     )
@@
       (effects (font (size 1.27 1.27)) hide)
     )
+    (property "JLCPCB_CORRECTION" "0;0;180" (id 6) (at 124.46 53.34 0)
+      (effects (font (size 1.27 1.27)) hide)
+    )
     (pin "1")
     (pin "2")
@@
       (effects (font (size 1.27 1.27)) hide)
     )
+    (property "JLCPCB_IGNORE" "1" (id 4) (at 269.24 91.44 0)
+      (effects (font (size 1.27 1.27)) hide)
+    )

Commit message: correction of USP-C footprint
Parts:
- B1: JLCPCB_CORRECTION (none) -> 0;0;90
- J32: JLCPCB_CORRECTION (none) -> 0;-1.27;90; LCSC 22284020 -> C234182
Changed lines of the file:
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@@
+      (effects (font (size 1.27 1.27)) hide)
+    )
+    (property "JLCPCB_CORRECTION" "0;0;90" (id 6) (at 134.62 48.26 0)
       (effects (font (size 1.27 1.27)) hide)
     )
@@
       (effects (font (size 1.27 1.27)) hide)
     )
-    (property "LCSC" "22284020" (id 4) (at 269.24 127 0)
+    (property "LCSC" "C234182" (id 4) (at 269.24 127 0)
       (effects (font (size 1.27 1.27)) hide)
     )
@@
       (effects (font (size 1.27 1.27)) hide)
     )
+    (property "JLCPCB_CORRECTION" "0;-1.27;90" (id 6) (at 269.24 127 0)
+      (effects (font (size 1.27 1.27)) hide)
+    )
