File: hw/RBCX_v1.3/Connectors.kicad_sch (KiCad schematic)
At the start: 82 parts

Commit message: Remove stepdowns, Micro-USB; fixup region names
Parts:
- D10: footprint (none) -> RBCX:SOD123
- D11: value (none) -> BAS40-05; footprint (none) -> RBCX:SOT23
- IM2: value (none) -> STEPDOWN; footprint (none) -> RBCX:STEPDOWN
- JP10: value (none) -> ESP_I2C_AUX1_VSEL; footprint (none) -> RBCX:1X03
- JP11: value (none) -> ESP_UART_AUX; footprint (none) -> RBCX:1X03
- JP12: value (none) -> ESP_SPI_AUX1; footprint (none) -> RBCX:1X03
- JP13: value (none) -> UTS2; footprint (none) -> RBCX:1X04
- JP14: value (none) -> ESP_I2C2_VSEL; footprint (none) -> RBCX:1X04
- JP15: value (none) -> ESP_SPI2; footprint (none) -> RBCX:1X06
- JP16: value (none) -> UTS3; footprint (none) -> RBCX:1X04
- JP17: value (none) -> ESP_I2C_AUX2_VSEL; footprint (none) -> RBCX:1X03
- JP18: value (none) -> STM_UART; footprint (none) -> RBCX:1X04
- JP19: value (none) -> ESP_SPI_AUX2; footprint (none) -> RBCX:1X03
- JP20: value (none) -> UTS4; footprint (none) -> RBCX:1X04
- JP21: value (none) -> ESP_SPI3; footprint (none) -> RBCX:1X06
- JP22: value (none) -> ESP_I2C1; footprint (none) -> RBCX:1X04
- JP23: value (none) -> ESP_UCOM; footprint (none) -> RBCX:1X04
- JP24: value (none) -> ESP_SPI_AUX3; footprint (none) -> RBCX:1X03
- JP25: value (none) -> ESP_I2C_AUX1; footprint (none) -> RBCX:1X03
- JP26: value (none) -> ESP_UCOM_AUX; footprint (none) -> RBCX:1X03
- JP27: value (none) -> ILED_EN; footprint (none) -> RBCX:1X01
- JP28: value (none) -> ESP_I2C2; footprint (none) -> RBCX:1X04
- JP29: value (none) -> AIO; footprint (none) -> RBCX:2X04
- JP30: value (none) -> ESP_I2C_AUX2; footprint (none) -> RBCX:1X03
- JP31: value (none) -> ILED; footprint (none) -> RBCX:1X03
- JP6: value (none) -> UTS1; footprint (none) -> RBCX:1X04
- JP7: value (none) -> ESP_I2C1_VSEL; footprint (none) -> RBCX:1X04
- JP8: value (none) -> ESP_SPI1; footprint (none) -> RBCX:1X06
- JP9: value (none) -> ESP_UART; footprint (none) -> RBCX:1X04
- Q5, Q6, Q7, Q8: footprint (none) -> RBCX:SOT23
- R24, R25, R37, R38, R42, R43, R50, R62, R64: value (none) -> 4k7; footprint (none) -> RBCX:R0402
- R26, R27, R28, R29, R30, R31, R32, R33, R34, R35, R36, R39, R40, R41, R44, R45, R46, R47, R48, R49, R52, R53, R54, R55, R56, R58, R59, R60, R61, R65: value (none) -> 330R; footprint (none) -> RBCX:R0402
- R51, R57: value (none) -> 100k; footprint (none) -> RBCX:R0402
- R63: value (none) -> 0R; footprint (none) -> RBCX:R1206
- SJ1, SJ2, SJ3, SJ4, SJ5: value (none) -> SJ2W_DEFAULT; footprint (none) -> RBCX:SJ_2_DEFAULT
- TP15, TP16: value (none) -> TP_06MM; footprint (none) -> RBCX:TP_06

Commit message: Everything everywhere all et once
Conversion to a new look
-  splitting the whole diagram for better orientation on multiple sheets using Kicad functions. Division of the whole schematics within several hierarchical sheets without globally named trac, using only wires, local labels and hierarchical labels.

Add new features
- Battery charger with cell balancer (With whole battery measurement)
- USB PD Sink Controller

Change old features
-  removing many 5V stepdowns and replacing them with only one strong stepdown (continuous 8A, peak 12A)
-  New power switcher design to connect VUSB to the VCC power line when no battery is connected.
(The reason for the new design is the implementation of Power deliveri => high voltage capability on VUSB 5-12V).

Remove micro_USB
Parts:
- removed D10: (no value), RBCX:SOD123, symbol RBCX-eagle-import:SHOTTKY-SOD123
- removed D11: BAS40-05, RBCX:SOT23, symbol RBCX-eagle-import:BAS40-05
- removed IM2: STEPDOWN, RBCX:STEPDOWN, symbol RBCX-eagle-import:STEPDOWN
- removed JP10: ESP_I2C_AUX1_VSEL, RBCX:1X03, symbol RBCX-eagle-import:PINHD-1X3
- removed JP11: ESP_UART_AUX, RBCX:1X03, symbol RBCX-eagle-import:PINHD-1X3
- removed JP12: ESP_SPI_AUX1, RBCX:1X03, symbol RBCX-eagle-import:PINHD-1X3
- removed JP13: UTS2, RBCX:1X04, symbol RBCX-eagle-import:PINHD-1X4
- removed JP14: ESP_I2C2_VSEL, RBCX:1X04, symbol RBCX-eagle-import:PINHD-1X4
- removed JP15: ESP_SPI2, RBCX:1X06, symbol RBCX-eagle-import:PINHD-1X6
- removed JP16: UTS3, RBCX:1X04, symbol RBCX-eagle-import:PINHD-1X4
- removed JP17: ESP_I2C_AUX2_VSEL, RBCX:1X03, symbol RBCX-eagle-import:PINHD-1X3
- removed JP18: STM_UART, RBCX:1X04, symbol RBCX-eagle-import:PINHD-1X4
- removed JP19: ESP_SPI_AUX2, RBCX:1X03, symbol RBCX-eagle-import:PINHD-1X3
- removed JP20: UTS4, RBCX:1X04, symbol RBCX-eagle-import:PINHD-1X4
- removed JP21: ESP_SPI3, RBCX:1X06, symbol RBCX-eagle-import:PINHD-1X6
- removed JP22: ESP_I2C1, RBCX:1X04, symbol RBCX-eagle-import:PINHD-1X4
- removed JP23: ESP_UCOM, RBCX:1X04, symbol RBCX-eagle-import:PINHD-1X4
- removed JP24: ESP_SPI_AUX3, RBCX:1X03, symbol RBCX-eagle-import:PINHD-1X3
- removed JP25: ESP_I2C_AUX1, RBCX:1X03, symbol RBCX-eagle-import:PINHD-1X3
- removed JP26: ESP_UCOM_AUX, RBCX:1X03, symbol RBCX-eagle-import:PINHD-1X3
- removed JP27: ILED_EN, RBCX:1X01, symbol RBCX-eagle-import:PINHD-1X1
- removed JP28: ESP_I2C2, RBCX:1X04, symbol RBCX-eagle-import:PINHD-1X4
- removed JP29: AIO, RBCX:2X04, symbol RBCX-eagle-import:PINHD-2X4
- removed JP30: ESP_I2C_AUX2, RBCX:1X03, symbol RBCX-eagle-import:PINHD-1X3
- removed JP31: ILED, RBCX:1X03, symbol RBCX-eagle-import:PINHD-1X3
- removed JP6: UTS1, RBCX:1X04, symbol RBCX-eagle-import:PINHD-1X4
- removed JP7: ESP_I2C1_VSEL, RBCX:1X04, symbol RBCX-eagle-import:PINHD-1X4
- removed JP8: ESP_SPI1, RBCX:1X06, symbol RBCX-eagle-import:PINHD-1X6
- removed JP9: ESP_UART, RBCX:1X04, symbol RBCX-eagle-import:PINHD-1X4
- removed Q5, Q6, Q7, Q8: (no value), RBCX:SOT23, symbol RBCX-eagle-import:N-MOSFET-SOT23-GSD
- removed R24, R25, R37, R38, R42, R43, R50, R62, R64: 4k7, RBCX:R0402, symbol RBCX-eagle-import:R-EU_R0402
- removed R26, R27, R28, R29, R30, R31, R32, R33, R34, R35, R36, R39, R40, R41, R44, R45, R46, R47, R48, R49, R52, R53, R54, R55, R56, R58, R59, R60, R61, R65: 330R, RBCX:R0402, symbol RBCX-eagle-import:R-EU_R0402
- removed R51, R57: 100k, RBCX:R0402, symbol RBCX-eagle-import:R-EU_R0402
- removed R63: 0R, RBCX:R1206, symbol RBCX-eagle-import:R-EU_R1206
- removed SJ1, SJ2, SJ3, SJ4, SJ5: SJ2W_DEFAULT, RBCX:SJ_2_DEFAULT, symbol RBCX-eagle-import:SJ2W_DEFAULT
- removed TP15, TP16: TP_06MM, RBCX:TP_06, symbol RBCX-eagle-import:TP_06MM
- added D?: D, Diode_SMD:D_SOD-523, symbol Device:D
- added J? (x10): Conn_01x03, Connector_PinHeader_2.54mm:PinHeader_1x03_P2.54mm_Vertical, symbol Connector_Generic:Conn_01x03
- added J? (x6): Conn_01x04, Connector_PinHeader_2.54mm:PinHeader_1x04_P2.54mm_Vertical, symbol Connector_Generic:Conn_01x04
- added J? (x3): Conn_01x06, Connector_PinHeader_2.54mm:PinHeader_1x06_P2.54mm_Vertical, symbol Connector_Generic:Conn_01x06
- added JP? (x4): SolderJumper_3_Bridged12, Jumper:SolderJumper-3_P1.3mm_Bridged12_RoundedPad1.0x1.5mm, symbol Jumper:SolderJumper_3_Bridged12
- added Q? (x4): Q_NMOS_DGS, Package_TO_SOT_SMD:SOT-723, symbol Device:Q_NMOS_DGS
- added R? (x8): 4k7, Resistor_SMD:R_0201_0603Metric, symbol Device:R
- added R? (x16): 330, Capacitor_SMD:C_0201_0603Metric, symbol Device:R
- added R? (x2): 100k, Capacitor_SMD:C_0201_0603Metric, symbol Device:R
- added R?: 10k, Capacitor_SMD:C_0201_0603Metric, symbol Device:R
- added TP?: TP_06MM, RBCX:TP_06MM, symbol RBCX-eagle-import:TP_06MM
Connections:
- net ESP-I2C-PWR: now also J?.1 (Pin_1), J?.1 (Pin_1), J?.3 (Pin_3), J?.3 (Pin_3), JP?.2 (C), R?.2, R?.2, R?.2
- net ESP-I2C-SCL-VSEL: now also J?.3 (Pin_3), J?.3 (Pin_3), Q?.1 (D), R?.1
- net ESP-I2C-SDA-VSEL: now also J?.4 (Pin_4), J?.4 (Pin_4), Q?.1 (D), R?.1
- net ESP-SPI-MISO: now also J?.4 (Pin_4), J?.4 (Pin_4), J?.4 (Pin_4), R?.2
- net ESP-SPI-MOSI: now also J?.3 (Pin_3), J?.3 (Pin_3), J?.3 (Pin_3), R?.2
- net ESP-SPI-SCK: now also J?.5 (Pin_5), J?.5 (Pin_5), J?.5 (Pin_5), R?.2
- net ESP-SPI-~{CS1}: now also J?.6 (Pin_6), R?.2
- net ESP-SPI-~{CS2}: now also J?.6 (Pin_6), R?.2
- net ESP-SPI-~{CS3}: now also J?.6 (Pin_6), R?.2
- net ESP-USART-RX: now also J?.3 (Pin_3), R?.2
- net ESP-USART-TX: now also J?.4 (Pin_4), R?.2
- net ESP_EN: now also Q?.2 (G)
- net ESP_SPI_PWR: now also J?.1 (Pin_1), JP?.2 (C)
- net ESP_UCOM_PWR: now also J?.1 (Pin_1), JP?.2 (C)
- net ESP_USART_PWR: now also J?.1 (Pin_1), JP?.2 (C)
- net GND: now also J?.2 (Pin_2), J?.2 (Pin_2), J?.2 (Pin_2), J?.2 (Pin_2), J?.2 (Pin_2), J?.2 (Pin_2), J?.2 (Pin_2), J?.2 (Pin_2), J?.2 (Pin_2), J?.2 (Pin_2), J?.2 (Pin_2), J?.2 (Pin_2), J?.2 (Pin_2), J?.2 (Pin_2), J?.2 (Pin_2), J?.2 (Pin_2), J?.2 (Pin_2), J?.2 (Pin_2), J?.3 (Pin_3)
- net GPIO-1: now also J?.1 (Pin_1), R?.2
- net GPIO-3: now also J?.3 (Pin_3), R?.2
- net GPIO-4: now also J?.4 (Pin_4), R?.2
- net GPIO-6: now also J?.1 (Pin_1), R?.2
- net GPIO-7: now also Q?.3 (S), R?.1, R?.2
- net GPIO1: now also R?.1
- net GPIO2: now also J?.1 (Pin_1)
- net GPIO3: now also R?.1
- net GPIO4: now also R?.1
- net GPIO5: now also R?.1
- net ILED: now also Q?.3 (S), R?.2, TP?.P$1 (TP)
- net ILED-5V: now also J?.1 (Pin_1), Q?.1 (D), R?.1
- net IN1: now also J?.1 (Pin_1), R?.1
- net IN2: now also J?.1 (Pin_1), R?.1
- net IN3: now also D?.2 (A), R?.1
- net IN3-5V: now also J?.1 (Pin_1), R?.2
- net IN4: now also J?.1 (Pin_1), R?.1
- net SPI_MISO: now also R?.1
- net SPI_MOSI: now also R?.1
- net SPI_SCK: now also R?.1
- net SPI_~{SS1}: now also R?.1
- net SPI_~{SS2}: now also R?.1
- net UART2_RX: now also R?.1
- net UART2_TX: now also R?.1
- new net: D?.1 (K), R?.1
- new net: J?.1 (Pin_1), R?.2
- new net 3V3: J?.1 (Pin_1), J?.1 (Pin_1), J?.1 (Pin_1), J?.1 (Pin_1), J?.3 (Pin_3), J?.3 (Pin_3), J?.3 (Pin_3), J?.3 (Pin_3), J?.3 (Pin_3), J?.3 (Pin_3), J?.3 (Pin_3), JP?.1 (A), JP?.1 (A), JP?.1 (A), JP?.3 (B), Q?.2 (G), Q?.2 (G), Q?.2 (G), R?.2, R?.2, R?.2, R?.2, R?.2, R?.2, R?.2
- new net 5V: J?.2 (Pin_2), JP?.1 (A), JP?.3 (B), JP?.3 (B), JP?.3 (B), R?.2
- new net GPIO-7-VSEL: J?.1 (Pin_1), Q?.1 (D), R?.1
- new net GPIO6: R?.1
- new net GPIO7: R?.1
- new net I2C_SCL-PULLUP: J?.3 (Pin_3), J?.3 (Pin_3), Q?.3 (S), R?.1
- new net I2C_SDA-PULLUP: J?.4 (Pin_4), J?.4 (Pin_4), Q?.3 (S), R?.1
- new net I_LED: R?.1
- new net SPI_~{SS3}: R?.1
Other:
- note added: "v1.3"
- note removed: "ILED"
- note removed: "UART"
- note removed: "ULTRASONIC RANGEFINDERS"
- note removed: "v1.2"

Commit message: Work in progress
Parts:
- gave numbers to parts that had none: 56
Connections:
- net GPIO-5: now also J10.1 (Pin_1), R27.2

Commit message: New PCB layout
some changes of schema:
- change PD sink AO33772 to AO33771
- remove power switch
Parts:
- J10, J11, J14, J15, J16, J19, J20, J21, J23, J8: footprint Connector_PinHeader_2.54mm:PinHeader_1x03_P2.54mm_Vertical -> RBCX:PinHeader_1x03_P2.54mm_Vertical
- J12, J18, J5: footprint Connector_PinHeader_2.54mm:PinHeader_1x06_P2.54mm_Vertical -> RBCX:PinHeader_1x06_P2.54mm_Vertical
- J13, J17, J22, J6, J7, J9: footprint Connector_PinHeader_2.54mm:PinHeader_1x04_P2.54mm_Vertical -> RBCX:PinHeader_1x04_P2.54mm_Vertical
Changed lines of the file:
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@@
       (effects (font (size 1.27 1.27)) (justify left))
     )
-    (property "Footprint" "Connector_PinHeader_2.54mm:PinHeader_1x03_P2.54mm_Vertical" (id 2) (at 106.68 85.09 0)
+    (property "Footprint" "RBCX:PinHeader_1x03_P2.54mm_Vertical" (id 2) (at 106.68 85.09 0)
       (effects (font (size 1.27 1.27)) hide)
     )
@@
       (effects (font (size 1.27 1.27)) (justify left))
     )
-    (property "Footprint" "Connector_PinHeader_2.54mm:PinHeader_1x03_P2.54mm_Vertical" (id 2) (at 271.78 149.86 0)
+    (property "Footprint" "RBCX:PinHeader_1x03_P2.54mm_Vertical" (id 2) (at 271.78 149.86 0)
       (effects (font (size 1.27 1.27)) hide)
     )
@@
       (effects (font (size 1.27 1.27)) (justify left))
     )
-    (property "Footprint" "Connector_PinHeader_2.54mm:PinHeader_1x04_P2.54mm_Vertical" (id 2) (at 106.68 129.54 0)
+    (property "Footprint" "RBCX:PinHeader_1x04_P2.54mm_Vertical" (id 2) (at 106.68 129.54 0)
       (effects (font (size 1.27 1.27)) hide)
     )
@@
       (effects (font (size 1.27 1.27)) (justify left))
     )
-    (property "Footprint" "Connector_PinHeader_2.54mm:PinHeader_1x06_P2.54mm_Vertical" (id 2) (at 187.96 129.54 0)
+    (property "Footprint" "RBCX:PinHeader_1x06_P2.54mm_Vertical" (id 2) (at 187.96 129.54 0)
       (effects (font (size 1.27 1.27)) hide)
     )
@@
       (effects (font (size 1.27 1.27)) (justify left))
     )
-    (property "Footprint" "Connector_PinHeader_2.54mm:PinHeader_1x03_P2.54mm_Vertical" (id 2) (at 187.96 106.68 0)
+    (property "Footprint" "RBCX:PinHeader_1x03_P2.54mm_Vertical" (id 2) (at 187.96 106.68 0)
       (effects (font (size 1.27 1.27)) hide)
     )
@@
       (effects (font (size 1.27 1.27)) (justify left))
     )
-    (property "Footprint" "Connector_PinHeader_2.54mm:PinHeader_1x03_P2.54mm_Vertical" (id 2) (at 106.68 179.07 0)
+    (property "Footprint" "RBCX:PinHeader_1x03_P2.54mm_Vertical" (id 2) (at 106.68 179.07 0)
       (effects (font (size 1.27 1.27)) hide)
     )
@@
       (effects (font (size 1.27 1.27)) (justify left))
     )
-    (property "Footprint" "Connector_PinHeader_2.54mm:PinHeader_1x03_P2.54mm_Vertical" (id 2) (at 187.96 149.86 0)
+    (property "Footprint" "RBCX:PinHeader_1x03_P2.54mm_Vertical" (id 2) (at 187.96 149.86 0)
       (effects (font (size 1.27 1.27)) hide)
     )
@@
       (effects (font (size 1.27 1.27)) (justify left))
     )
-    (property "Footprint" "Connector_PinHeader_2.54mm:PinHeader_1x04_P2.54mm_Vertical" (id 2) (at 271.78 45.72 0)
+    (property "Footprint" "RBCX:PinHeader_1x04_P2.54mm_Vertical" (id 2) (at 271.78 45.72 0)
       (effects (font (size 1.27 1.27)) hide)
     )
@@
       (effects (font (size 1.27 1.27)) (justify left))
     )
-    (property "Footprint" "Connector_PinHeader_2.54mm:PinHeader_1x06_P2.54mm_Vertical" (id 2) (at 187.96 85.09 0)
+    (property "Footprint" "RBCX:PinHeader_1x06_P2.54mm_Vertical" (id 2) (at 187.96 85.09 0)
       (effects (font (size 1.27 1.27)) hide)
     )
@@
       (effects (font (size 1.27 1.27)) (justify left))
     )
-    (property "Footprint" "Connector_PinHeader_2.54mm:PinHeader_1x04_P2.54mm_Vertical" (id 2) (at 106.68 162.56 0)
+    (property "Footprint" "RBCX:PinHeader_1x04_P2.54mm_Vertical" (id 2) (at 106.68 162.56 0)
       (effects (font (size 1.27 1.27)) hide)
     )
@@
       (effects (font (size 1.27 1.27)) (justify left))
     )
-    (property "Footprint" "Connector_PinHeader_2.54mm:PinHeader_1x03_P2.54mm_Vertical" (id 2) (at 106.68 104.14 0)
+    (property "Footprint" "RBCX:PinHeader_1x03_P2.54mm_Vertical" (id 2) (at 106.68 104.14 0)
       (effects (font (size 1.27 1.27)) hide)
     )
@@
       (effects (font (size 1.27 1.27)) (justify left))
     )
-    (property "Footprint" "Connector_PinHeader_2.54mm:PinHeader_1x03_P2.54mm_Vertical" (id 2) (at 187.96 58.42 0)
+    (property "Footprint" "RBCX:PinHeader_1x03_P2.54mm_Vertical" (id 2) (at 187.96 58.42 0)
       (effects (font (size 1.27 1.27)) hide)
     )
@@
       (effects (font (size 1.27 1.27)) (justify left))
     )
-    (property "Footprint" "Connector_PinHeader_2.54mm:PinHeader_1x04_P2.54mm_Vertical" (id 2) (at 106.68 40.64 0)
+    (property "Footprint" "RBCX:PinHeader_1x04_P2.54mm_Vertical" (id 2) (at 106.68 40.64 0)
       (effects (font (size 1.27 1.27)) hide)
     )
@@
       (effects (font (size 1.27 1.27)) (justify left))
     )
-    (property "Footprint" "Connector_PinHeader_2.54mm:PinHeader_1x03_P2.54mm_Vertical" (id 2) (at 271.78 109.22 0)
+    (property "Footprint" "RBCX:PinHeader_1x03_P2.54mm_Vertical" (id 2) (at 271.78 109.22 0)
       (effects (font (size 1.27 1.27)) hide)
     )
@@
       (effects (font (size 1.27 1.27)) (justify left))
     )
-    (property "Footprint" "Connector_PinHeader_2.54mm:PinHeader_1x03_P2.54mm_Vertical" (id 2) (at 106.68 147.32 0)
+    (property "Footprint" "RBCX:PinHeader_1x03_P2.54mm_Vertical" (id 2) (at 106.68 147.32 0)
       (effects (font (size 1.27 1.27)) hide)
     )
@@
       (effects (font (size 1.27 1.27)) (justify left))
     )
-    (property "Footprint" "Connector_PinHeader_2.54mm:PinHeader_1x03_P2.54mm_Vertical" (id 2) (at 271.78 63.5 0)
+    (property "Footprint" "RBCX:PinHeader_1x03_P2.54mm_Vertical" (id 2) (at 271.78 63.5 0)
       (effects (font (size 1.27 1.27)) hide)
     )
@@
       (effects (font (size 1.27 1.27)) (justify left))
     )
-    (property "Footprint" "Connector_PinHeader_2.54mm:PinHeader_1x06_P2.54mm_Vertical" (id 2) (at 187.96 38.1 0)
+    (property "Footprint" "RBCX:PinHeader_1x06_P2.54mm_Vertical" (id 2) (at 187.96 38.1 0)
       (effects (font (size 1.27 1.27)) hide)
     )
@@
       (effects (font (size 1.27 1.27)) (justify left))
     )
-    (property "Footprint" "Connector_PinHeader_2.54mm:PinHeader_1x04_P2.54mm_Vertical" (id 2) (at 271.78 90.17 0)
+    (property "Footprint" "RBCX:PinHeader_1x04_P2.54mm_Vertical" (id 2) (at 271.78 90.17 0)
       (effects (font (size 1.27 1.27)) hide)
     )
@@
       (effects (font (size 1.27 1.27)) (justify left))
     )
-    (property "Footprint" "Connector_PinHeader_2.54mm:PinHeader_1x04_P2.54mm_Vertical" (id 2) (at 106.68 63.5 0)
-      (effects (font (size 1.27 1.27)) hide)
-    )
+    (property "Footprint" "RBCX:PinHeader_1x04_P2.54mm_Vertical" (id 2) (at 106.68 63.5 0)
+      (effects (font (size 1.27 1.27)) hide)
+    )

Commit message: Production files
Parts:
- J10, J11, J14, J15, J16, J19, J20, J21, J23, J8: JLCPCB_CORRECTION (none) -> 0;-2.54;90
- J12, J18, J5: JLCPCB_CORRECTION (none) -> 0;-6.35;90
- J13, J17, J22, J6, J7, J9: JLCPCB_CORRECTION (none) -> 0;-3.81;90
- Q1, Q2, Q3, Q4: JLCPCB_CORRECTION (none) -> 0;0;180
- TP9: JLCPCB_IGNORE (none) -> 1
Changed lines of the file:
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@@
+      (effects (font (size 1.27 1.27)) hide)
+    )
+    (property "JLCPCB_CORRECTION" "0;-2.54;90" (id 6) (at 106.68 85.09 0)
       (effects (font (size 1.27 1.27)) hide)
     )
@@
       (effects (font (size 1.27 1.27)) hide)
     )
+    (property "JLCPCB_CORRECTION" "0;0;180" (id 6) (at 60.96 91.44 0)
+      (effects (font (size 1.27 1.27)) hide)
+    )
     (pin "1")
     (pin "2")
@@
     )
     (property "Basic/Extended" "E" (id 5) (at 271.78 149.86 0)
+      (effects (font (size 1.27 1.27)) hide)
+    )
+    (property "JLCPCB_CORRECTION" "0;-2.54;90" (id 6) (at 271.78 149.86 0)
       (effects (font (size 1.27 1.27)) hide)
     )
@@
       (effects (font (size 1.27 1.27)) hide)
     )
+    (property "JLCPCB_CORRECTION" "0;-3.81;90" (id 6) (at 106.68 129.54 0)
+      (effects (font (size 1.27 1.27)) hide)
+    )
     (pin "1")
     (pin "2")
@@
     )
     (property "Basic/Extended" "E" (id 5) (at 187.96 129.54 0)
+      (effects (font (size 1.27 1.27)) hide)
+    )
+    (property "JLCPCB_CORRECTION" "0;-6.35;90" (id 6) (at 187.96 129.54 0)
       (effects (font (size 1.27 1.27)) hide)
     )
@@
       (effects (font (size 1.27 1.27)) hide)
     )
+    (property "JLCPCB_CORRECTION" "0;0;180" (id 6) (at 240.03 144.78 0)
+      (effects (font (size 1.27 1.27)) hide)
+    )
     (pin "1")
     (pin "2")
@@
       (effects (font (size 1.27 1.27)) hide)
     )
+    (property "JLCPCB_CORRECTION" "0;-2.54;90" (id 6) (at 187.96 106.68 0)
+      (effects (font (size 1.27 1.27)) hide)
+    )
     (pin "1")
     (pin "2")
@@
     )
     (property "Basic/Extended" "E" (id 5) (at 106.68 179.07 0)
+      (effects (font (size 1.27 1.27)) hide)
+    )
+    (property "JLCPCB_CORRECTION" "0;-2.54;90" (id 6) (at 106.68 179.07 0)
       (effects (font (size 1.27 1.27)) hide)
     )
@@
       (effects (font (size 1.27 1.27)) hide)
     )
+    (property "JLCPCB_CORRECTION" "0;0;180" (id 6) (at 60.96 66.04 0)
+      (effects (font (size 1.27 1.27)) hide)
+    )
     (pin "1")
     (pin "2")
@@
       (effects (font (size 1.27 1.27)) hide)
     )
+    (property "JLCPCB_CORRECTION" "0;-2.54;90" (id 6) (at 187.96 149.86 0)
+      (effects (font (size 1.27 1.27)) hide)
+    )
     (pin "1")
     (pin "2")
@@
       (effects (font (size 1.27 1.27)) hide)
     )
+    (property "JLCPCB_CORRECTION" "0;-3.81;90" (id 6) (at 271.78 45.72 0)
+      (effects (font (size 1.27 1.27)) hide)
+    )
     (pin "1")
     (pin "2")
@@
       (effects (font (size 1.27 1.27)) hide)
     )
+    (property "JLCPCB_CORRECTION" "0;-6.35;90" (id 6) (at 187.96 85.09 0)
+      (effects (font (size 1.27 1.27)) hide)
+    )
     (pin "1")
     (pin "2")
@@
       (effects (font (size 1.27 1.27)) hide)
     )
+    (property "JLCPCB_CORRECTION" "0;-3.81;90" (id 6) (at 106.68 162.56 0)
+      (effects (font (size 1.27 1.27)) hide)
+    )
     (pin "1")
     (pin "2")
@@
     )
     (property "Basic/Extended" "E" (id 5) (at 106.68 104.14 0)
+      (effects (font (size 1.27 1.27)) hide)
+    )
+    (property "JLCPCB_CORRECTION" "0;-2.54;90" (id 6) (at 106.68 104.14 0)
       (effects (font (size 1.27 1.27)) hide)
     )
@@
       (effects (font (size 1.27 1.27)) hide)
     )
+    (property "JLCPCB_CORRECTION" "0;-2.54;90" (id 6) (at 187.96 58.42 0)
+      (effects (font (size 1.27 1.27)) hide)
+    )
     (pin "1")
     (pin "2")
@@
       (effects (font (size 1.27 1.27)) hide)
     )
+    (property "JLCPCB_CORRECTION" "0;-3.81;90" (id 6) (at 106.68 40.64 0)
+      (effects (font (size 1.27 1.27)) hide)
+    )
     (pin "1")
     (pin "2")
@@
     )
     (property "Basic/Extended" "E" (id 5) (at 271.78 109.22 0)
+      (effects (font (size 1.27 1.27)) hide)
+    )
+    (property "JLCPCB_CORRECTION" "0;-2.54;90" (id 6) (at 271.78 109.22 0)
       (effects (font (size 1.27 1.27)) hide)
     )
@@
       (effects (font (size 1.27 1.27)) hide)
     )
+    (property "JLCPCB_CORRECTION" "0;0;180" (id 6) (at 60.96 40.64 0)
+      (effects (font (size 1.27 1.27)) hide)
+    )
     (pin "1")
     (pin "2")
@@
       (effects (font (size 1.27 1.27)) hide)
     )
+    (property "JLCPCB_CORRECTION" "0;-2.54;90" (id 6) (at 106.68 147.32 0)
+      (effects (font (size 1.27 1.27)) hide)
+    )
     (pin "1")
     (pin "2")
@@
     )
     (property "Basic/Extended" "E" (id 5) (at 271.78 63.5 0)
+      (effects (font (size 1.27 1.27)) hide)
+    )
+    (property "JLCPCB_CORRECTION" "0;-2.54;90" (id 6) (at 271.78 63.5 0)
       (effects (font (size 1.27 1.27)) hide)
     )
@@
       (effects (font (size 1.27 1.27)) hide)
     )
+    (property "JLCPCB_CORRECTION" "0;-6.35;90" (id 6) (at 187.96 38.1 0)
+      (effects (font (size 1.27 1.27)) hide)
+    )
     (pin "1")
     (pin "2")
@@
       (effects (font (size 1.27 1.27)) hide)
     )
+    (property "JLCPCB_CORRECTION" "0;-3.81;90" (id 6) (at 271.78 90.17 0)
+      (effects (font (size 1.27 1.27)) hide)
+    )
     (pin "1")
     (pin "2")
@@
       (effects (font (size 1.27 1.27)) hide)
     )
+    (property "JLCPCB_CORRECTION" "0;-3.81;90" (id 6) (at 106.68 63.5 0)
+      (effects (font (size 1.27 1.27)) hide)
+    )
     (pin "1")
     (pin "2")
@@
       (effects (font (size 1.27 1.27)) hide)
     )
+    (property "JLCPCB_IGNORE" "1" (id 4) (at 232.41 149.86 0)
+      (effects (font (size 1.27 1.27)) hide)
+    )

Commit message: Kuba issues
Change of power transistor from JSM3622 to JMSL0302AU

NTC connectors

Moving the Cell balancer behind the switch

and some little things
Changed lines of the file:
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@@
   )
   (text "IO12/TDI on ESP32 has internal pull-down\nduring releasing EN, so we need to switch-off\nthe transistor to disconnect pull/up R64."
-    (at 147.32 181.61 180)
+    (at 237.49 142.24 180)
     (effects (font (size 1.27 1.0795)) (justify right bottom))
   )
@@
   (symbol (lib_id "Device:R") (at 226.06 147.32 90) (unit 1)
     (in_bom yes) (on_board yes)
-    (property "Reference" "R43" (id 0) (at 226.06 142.24 90))
-    (property "Value" "330" (id 1) (at 226.06 144.78 90))
+    (property "Reference" "R43" (id 0) (at 228.6 149.86 90))
+    (property "Value" "330" (id 1) (at 222.25 149.86 90))
     (property "Footprint" "Capacitor_SMD:C_0201_0603Metric" (id 2) (at 226.06 149.098 90)
       (effects (font (size 1.27 1.27)) hide)
