File: hw/RBCX_v1.3/RBCX.kicad_sch (KiCad schematic)
At the start: 13 parts, among them J1 Conn_02x02_Odd_Even

Commit message: USB-DET level shifter
Parts:
- removed R159: 10k, Capacitor_SMD:C_0201_0603Metric, symbol Device:R
Changed lines of the file:
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@@
 (kicad_sch (version 20211123) (generator eeschema)
   (paper "A3")
-  (junction (at 147.32 68.58) (diameter 0) (color 0 0 0 0)
-  )
   (junction (at 267.97 148.59) (diameter 0) (color 255 136 0 1)
   )
@@
   (junction (at 267.97 104.14) (diameter 0) (color 255 136 0 1)
   )
-  (junction (at 144.78 50.8) (diameter 0) (color 255 153 0 1)
-  )
   (junction (at 220.98 100.33) (diameter 0) (color 0 0 0 0)
   )
@@
     (stroke (width 0) (type dash_dot) (color 0 136 255 1))
   )
-  (wire (pts (xy 147.32 50.8) (xy 144.78 50.8))
-    (stroke (width 0) (type default) (color 255 153 0 1))
-  )
   (wire (pts (xy 203.2 246.38) (xy 226.06 246.38))
     (stroke (width 0) (type default) (color 0 0 0 0))
@@
     (stroke (width 0) (type default) (color 0 0 0 0))
   )
-  (wire (pts (xy 139.7 68.58) (xy 147.32 68.58))
+  (wire (pts (xy 139.7 68.58) (xy 165.1 68.58))
     (stroke (width 0) (type default) (color 0 0 0 0))
   )
@@
     (stroke (width 0) (type default) (color 0 0 0 0))
   )
-  (wire (pts (xy 147.32 60.96) (xy 147.32 68.58))
-    (stroke (width 0) (type default) (color 0 0 0 0))
-  )
   (wire (pts (xy 93.98 182.88) (xy 165.1 182.88))
     (stroke (width 0) (type default) (color 0 0 0 0))
@@
     (stroke (width 0) (type default) (color 0 0 0 0))
   )
-  (wire (pts (xy 147.32 53.34) (xy 147.32 50.8))
-    (stroke (width 0) (type default) (color 255 153 0 1))
-  )
   (wire (pts (xy 78.74 25.4) (xy 78.74 52.07))
     (stroke (width 0) (type default) (color 255 0 0 1))
@@
     (stroke (width 0) (type default) (color 0 0 0 0))
   )
-  (wire (pts (xy 144.78 50.8) (xy 144.78 106.68))
-    (stroke (width 0) (type default) (color 255 136 0 1))
-  )
   (wire (pts (xy 336.55 80.01) (xy 344.17 80.01))
     (stroke (width 0) (type default) (color 0 0 0 0))
@@
     (stroke (width 0) (type default) (color 0 0 0 0))
   )
-  (wire (pts (xy 147.32 68.58) (xy 165.1 68.58))
-    (stroke (width 0) (type default) (color 0 0 0 0))
-  )
   (wire (pts (xy 257.81 148.59) (xy 267.97 148.59))
     (stroke (width 0) (type default) (color 255 136 0 1))
   )
-  (wire (pts (xy 144.78 35.56) (xy 144.78 50.8))
+  (wire (pts (xy 144.78 35.56) (xy 144.78 106.68))
     (stroke (width 0) (type default) (color 255 136 0 1))
   )
@@
     (pin "1")
   )
-  (symbol (lib_id "Device:R") (at 147.32 57.15 180) (unit 1)
-    (in_bom yes) (on_board yes)
-    (property "Reference" "R159" (id 0) (at 151.13 58.42 0))
-    (property "Value" "10k" (id 1) (at 151.13 55.88 0))
-    (property "Footprint" "Capacitor_SMD:C_0201_0603Metric" (id 2) (at 149.098 57.15 90)
-      (effects (font (size 1.27 1.27)) hide)
-    )
-    (property "Datasheet" "~" (id 3) (at 147.32 57.15 0)
-      (effects (font (size 1.27 1.27)) hide)
-    )
-    (property "LCSC" "C106225" (id 4) (at 147.32 57.15 0)
-      (effects (font (size 1.27 1.27)) hide)
-    )
-    (property "Basic/Extended" "E" (id 5) (at 147.32 57.15 0)
-      (effects (font (size 1.27 1.27)) hide)
-    )
-    (pin "1")
-    (pin "2")
-  )
   (symbol (lib_id "power:GND") (at 111.76 166.37 0) (unit 1)
     (in_bom yes) (on_board yes) (fields_autoplaced)
@@
       (reference "C84") (unit 1) (value "100nF") (footprint "Capacitor_SMD:C_0402_1005Metric")
     )
+    (path "/6bbf37d2-9f87-4f2b-9e95-56d617eb6363/f8a0606d-c386-4d1f-813a-fe76fb28f2a2"
+      (reference "C?") (unit 1) (value "C_Polarized") (footprint "Capacitor_SMD:CP_Elec_8x11.9")
+    )
     (path "/475071ea-f096-4c42-885f-4369ed96d957/f7bde2a5-9bdd-4058-808b-f32fc1b0fba0"
       (reference "D1") (unit 1) (value "D") (footprint "Diode_SMD:D_SOD-523")
@@
       (reference "D25") (unit 1) (value "D_Schottky") (footprint "Diode_SMD:D_SOD-123F")
     )
-    (path "/10e93c09-17c0-4b9f-b76a-d2803ee0aa4b/d1857828-09a5-429c-adc4-eb63905da129"
-      (reference "D26") (unit 1) (value "D") (footprint "Diode_SMD:D_SOD-523")
-    )
     (path "/6bbf37d2-9f87-4f2b-9e95-56d617eb6363/c6773705-1703-4f22-9161-c5523121e6c3"
       (reference "D27") (unit 1) (value "red") (footprint "LED_SMD:LED_0603_1608Metric")
@@
       (reference "Q14") (unit 1) (value "Q_PMOS_DGS") (footprint "RBCX:JMSL0302AU")
     )
+    (path "/10e93c09-17c0-4b9f-b76a-d2803ee0aa4b/f0000c14-40ba-4db4-b66b-dfb55f8c0b18"
+      (reference "Q15") (unit 1) (value "Q_NMOS_DGS") (footprint "Package_TO_SOT_SMD:SOT-723")
+    )
     (path "/69d4b832-77c1-4ad5-b705-7e6e572992c7"
       (reference "R1") (unit 1) (value "330") (footprint "Capacitor_SMD:C_0201_0603Metric")
@@
       (reference "R158") (unit 1) (value "10k") (footprint "Capacitor_SMD:C_0201_0603Metric")
     )
-    (path "/5c580c13-9983-40b7-8356-46c82dd64f7c"
-      (reference "R159") (unit 1) (value "10k") (footprint "Capacitor_SMD:C_0201_0603Metric")
+    (path "/10e93c09-17c0-4b9f-b76a-d2803ee0aa4b/8e9a9666-5b65-4c6b-b6f3-1f1c47ea29fc"
+      (reference "R159") (unit 1) (value "100k") (footprint "Capacitor_SMD:C_0201_0603Metric")
     )
     (path "/6bbf37d2-9f87-4f2b-9e95-56d617eb6363/72bdaae6-b602-4afd-90f1-5faa6da77e38/4bb0b1cf-522e-41ad-bcfb-369bcea14ef0"
