File: hw/RBCX_v1.3/Servos.kicad_sch (KiCad schematic)
At the start: 76 parts

Commit message: Remove stepdowns, Micro-USB; fixup region names
Parts:
- removed D27, D28: (no value), symbol RBCX-eagle-import:BAS40-05
- removed IM5, IM6, IM7, IM8: (no value), symbol RBCX-eagle-import:STEPDOWN
- removed JP48, JP49, JP50, JP51: (no value), symbol RBCX-eagle-import:PINHD-1X1
- removed R128, R129, R130, R131: (no value), symbol RBCX-eagle-import:R-EU_R1206
- C24, C25, C26, C27, C40: footprint (none) -> RBCX:E5-10,5
- C28, C29, C30, C31, C32, C33, C34, C35: footprint (none) -> RBCX:C0402
- C36, C37, C38, C39: footprint (none) -> RBCX:C0805
- D29, D30, D31, D32: value (none) -> SS34; footprint (none) -> RBCX:SMA
- D33, D34, D35, D36, D37: value (none) -> BAS40-04; footprint (none) -> RBCX:SOT23
- IC10, IC11, IC8, IC9: footprint (none) -> RBCX:SOT23-5L
- JP52: value (none) -> SERVO1; footprint (none) -> RBCX:1X03
- JP53: value (none) -> SERVO2; footprint (none) -> RBCX:1X03
- JP54: value (none) -> SERVO3; footprint (none) -> RBCX:1X03
- JP55: value (none) -> SERVO4; footprint (none) -> RBCX:1X03
- JP56, JP57: footprint (none) -> RBCX:JST-PH3
- R132, R134, R136, R138: value (none) -> 1k; footprint (none) -> RBCX:R0402
- R133, R135, R137, R139: footprint (none) -> RBCX:R1206
- R140, R141, R142, R143, R144: value (none) -> 2k2; footprint (none) -> RBCX:R0402
- TP46, TP47, TP48, TP49, TP50, TP51, TP52, TP53, TP54, TP55, TP56, TP57, TP58: value (none) -> TP_06MM; footprint (none) -> RBCX:TP_06
Connections:
- net SERVO1PWR is gone; now on net +5V: D29.A
- net SERVO2PWR is gone; now on net +5V: D30.A
- net SERVO3PWR is gone; now on net +5V: D31.A
- net SERVO4PWR is gone; now on net +5V: D32.A

Commit message: Everything everywhere all et once
Conversion to a new look
-  splitting the whole diagram for better orientation on multiple sheets using Kicad functions. Division of the whole schematics within several hierarchical sheets without globally named trac, using only wires, local labels and hierarchical labels.

Add new features
- Battery charger with cell balancer (With whole battery measurement)
- USB PD Sink Controller

Change old features
-  removing many 5V stepdowns and replacing them with only one strong stepdown (continuous 8A, peak 12A)
-  New power switcher design to connect VUSB to the VCC power line when no battery is connected.
(The reason for the new design is the implementation of Power deliveri => high voltage capability on VUSB 5-12V).

Remove micro_USB
Parts:
- removed C24, C25, C26, C27, C40: (no value), RBCX:E5-10,5, symbol RBCX-eagle-import:CPOL-EUE5-10.5
- removed C28, C29, C30, C31, C32, C33, C34, C35: (no value), RBCX:C0402, symbol RBCX-eagle-import:C-EUC0402
- removed C36, C37, C38, C39: (no value), RBCX:C0805, symbol RBCX-eagle-import:C-EUC0805
- removed D29, D30, D31, D32: SS34, RBCX:SMA, symbol RBCX-eagle-import:SHOTTKY-SMA
- removed D33, D34, D35, D36, D37: BAS40-04, RBCX:SOT23, symbol RBCX-eagle-import:BAS40-04
- removed IC10, IC11, IC8, IC9: (no value), RBCX:SOT23-5L, symbol RBCX-eagle-import:INA180A
- removed JP52: SERVO1, RBCX:1X03, symbol RBCX-eagle-import:PINHD-1X3
- removed JP53: SERVO2, RBCX:1X03, symbol RBCX-eagle-import:PINHD-1X3
- removed JP54: SERVO3, RBCX:1X03, symbol RBCX-eagle-import:PINHD-1X3
- removed JP55: SERVO4, RBCX:1X03, symbol RBCX-eagle-import:PINHD-1X3
- removed JP56, JP57: (no value), RBCX:JST-PH3, symbol RBCX-eagle-import:JST-PH3
- removed R132, R134, R136, R138: 1k, RBCX:R0402, symbol RBCX-eagle-import:R-EU_R0402
- removed R133, R135, R137, R139: (no value), RBCX:R1206, symbol RBCX-eagle-import:R-EU_R1206
- removed R140, R141, R142, R143, R144: 2k2, RBCX:R0402, symbol RBCX-eagle-import:R-EU_R0402
- removed TP46, TP47, TP48, TP49, TP50, TP51, TP52, TP53, TP54, TP55, TP56, TP57, TP58: TP_06MM, RBCX:TP_06, symbol RBCX-eagle-import:TP_06MM
- added C?: 220uF, Capacitor_SMD:CP_Elec_8x11.9, symbol Device:C_Polarized
- added D?: BAT54S, Package_TO_SOT_SMD:SOT-23, symbol RBCX:BAT54S
- added JP? (x2): (no value), RBCX:JST-PH3, symbol RBCX-eagle-import:JST-PH3
- added R?: 2.2k, Resistor_SMD:R_0201_0603Metric, symbol Device:R
- added TP?: TP_06MM, RBCX:TP_06MM, symbol RBCX-eagle-import:TP_06MM
Connections:
- net GND: now also C?.1, C?.2, D?.2 (A2), JP?.1, JP?.1, JP?.2, JP?.2, JP?.3, JP?.3, R?.1
- net INTELLIGENT_SERVO: now also D?.3 (C), R?.2, TP?.P$1 (TP)
- new net 3V3: D?.1 (A1)
Other:
- added sheet Classic Sevo 1 (Classic_sevo.kicad_sch)
- added sheet Classic Sevo 2 (Classic_sevo.kicad_sch)
- added sheet Classic Sevo 3 (Classic_sevo.kicad_sch)
- added sheet Classic Sevo 4 (Classic_sevo.kicad_sch)
- note added: "v1.3"
- note removed: "Fmax = 160 Hz"
- note removed: "v1.2"

Commit message: Work in progress
Parts:
- D23: renamed from D?; footprint Package_TO_SOT_SMD:SOT-23 -> Package_TO_SOT_SMD:SOT-523; LCSC C2828465 -> C134414
- gave numbers to parts that had none: 5

Commit message: Production files
Parts:
- D23: JLCPCB_CORRECTION (none) -> 0;0;180
- TP52: JLCPCB_IGNORE (none) -> 1
Changed lines of the file:
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@@
+      (effects (font (size 1.27 1.27)) hide)
+    )
+    (property "JLCPCB_IGNORE" "1" (id 4) (at 111.76 44.45 0)
       (effects (font (size 1.27 1.27)) hide)
     )
@@
       (effects (font (size 1.27 1.27)) hide)
     )
+    (property "JLCPCB_CORRECTION" "0;0;180" (id 6) (at 123.19 46.99 0)
+      (effects (font (size 1.27 1.27)) hide)
+    )

Commit message: ESD and I-Servo hacker
Parts:
- added TP?: TP_06MM, RBCX:TP_06MM, symbol RBCX-eagle-import:TP_06MM
Connections:
- net GND: now also TP?.P$1 (TP)
Changed lines of the file:
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@@
+    (stroke (width 0) (type default) (color 0 0 0 0))
+  )
+  (wire (pts (xy 148.59 44.45) (xy 148.59 46.99))
     (stroke (width 0) (type default) (color 0 0 0 0))
   )
@@
     (pin "3")
   )
+  (symbol (lib_id "RBCX-eagle-import:TP_06MM") (at 148.59 44.45 0) (unit 1)
+    (in_bom yes) (on_board yes)
+    (property "Reference" "TP?" (id 0) (at 146.05 36.83 0)
+      (effects (font (size 1.778 1.5113)) (justify left bottom))
+    )
+    (property "Value" "TP_06MM" (id 1) (at 146.05 39.116 0)
+      (effects (font (size 1.778 1.5113)) (justify left bottom))
+    )
+    (property "Footprint" "RBCX:TP_06MM" (id 2) (at 148.59 44.45 0)
+      (effects (font (size 1.27 1.27)) hide)
+    )
+    (property "Datasheet" "" (id 3) (at 148.59 44.45 0)
+      (effects (font (size 1.27 1.27)) hide)
+    )
+    (property "JLCPCB_IGNORE" "1" (id 4) (at 148.59 44.45 0)
+      (effects (font (size 1.27 1.27)) hide)
+    )
+    (pin "P$1")
+  )
   (symbol (lib_id "Device:R") (at 129.54 46.99 270) (unit 1)
